File: Microphone board/EEPROM.kicad_sch (KiCad schematic)
At the start: 1 part, among them U2 24LC256

Commit message: Made almost the rest of the schematic lol
Parts:
- added C69: 100n, Capacitor_SMD:C_0402_1005Metric, symbol Device:C
Connections:
- net GND: now reaches U2.1 (A0)
- net GND: now also U2.2 (A1), U2.3 (A2), U2.4 (GND), U2.7 (WP), C69.2
- net SDA: now reaches U2.5 (SDA)
- net SCL: now reaches U2.6 (SCL)
- net +3V3: now reaches U2.8 (VCC)
- net +3V3: now also C69.1

Commit message: almost finished power
Parts:
- renumbered C69 to C40
Changed lines of the file:
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@@
 		(dnp no)
 		(fields_autoplaced yes)
-		(property "Reference" "#PWR069"
+		(property "Reference" "#PWR029"
 			(at 146.05 93.98 0)
 			(hide yes)
@@
 			(project "Microphone board"
 				(path "/54b36551-a175-45db-a91c-236f7d72a35b/5745e146-afc6-45b9-a117-0cabb33abc50"
-					(reference "#PWR069")
+					(reference "#PWR029")
 					(unit 1)
 				)
@@
 		(dnp no)
 		(fields_autoplaced yes)
-		(property "Reference" "#PWR0106"
+		(property "Reference" "#PWR027"
 			(at 115.57 110.49 0)
 			(hide yes)
@@
 			(project "Microphone board"
 				(path "/54b36551-a175-45db-a91c-236f7d72a35b/5745e146-afc6-45b9-a117-0cabb33abc50"
-					(reference "#PWR0106")
+					(reference "#PWR027")
 					(unit 1)
 				)
@@
 		(dnp no)
 		(fields_autoplaced yes)
-		(property "Reference" "#PWR072"
+		(property "Reference" "#PWR031"
 			(at 158.75 116.84 0)
 			(hide yes)
@@
 			(project "Microphone board"
 				(path "/54b36551-a175-45db-a91c-236f7d72a35b/5745e146-afc6-45b9-a117-0cabb33abc50"
-					(reference "#PWR072")
+					(reference "#PWR031")
 					(unit 1)
 				)
@@
 		(dnp no)
 		(fields_autoplaced yes)
-		(property "Reference" "#PWR070"
+		(property "Reference" "#PWR030"
 			(at 146.05 116.84 0)
 			(hide yes)
@@
 			(project "Microphone board"
 				(path "/54b36551-a175-45db-a91c-236f7d72a35b/5745e146-afc6-45b9-a117-0cabb33abc50"
-					(reference "#PWR070")
+					(reference "#PWR030")
 					(unit 1)
 				)
@@
 		(dnp no)
 		(fields_autoplaced yes)
-		(property "Reference" "#PWR0107"
+		(property "Reference" "#PWR026"
 			(at 115.57 95.25 0)
 			(hide yes)
@@
 			(project "Microphone board"
 				(path "/54b36551-a175-45db-a91c-236f7d72a35b/5745e146-afc6-45b9-a117-0cabb33abc50"
-					(reference "#PWR0107")
+					(reference "#PWR026")
 					(unit 1)
 				)
@@
 		(dnp no)
 		(fields_autoplaced yes)
-		(property "Reference" "#PWR071"
+		(property "Reference" "#PWR028"
 			(at 133.35 116.84 0)
 			(hide yes)
@@
 			(project "Microphone board"
 				(path "/54b36551-a175-45db-a91c-236f7d72a35b/5745e146-afc6-45b9-a117-0cabb33abc50"
-					(reference "#PWR071")
+					(reference "#PWR028")
 					(unit 1)
 				)
@@
 		(dnp no)
 		(fields_autoplaced yes)
-		(property "Reference" "C69"
+		(property "Reference" "C40"
 			(at 119.38 96.5199 0)
 			(show_name no)
@@
 			(project "Microphone board"
 				(path "/54b36551-a175-45db-a91c-236f7d72a35b/5745e146-afc6-45b9-a117-0cabb33abc50"
-					(reference "C69")
-					(unit 1)
-				)
+					(reference "C40")
+					(unit 1)
+				)
