File: Microphone board/Microphone board.kicad_sch (KiCad schematic)
At the start: 0 parts

Commit message: Made almost the rest of the schematic lol
Other:
- sheet Trigger renamed User interface
- added sheet Power (power.kicad_sch)
- added sheet SD (SD.kicad_sch)
- added sheet USB (usb.kicad_sch)
- sheet Camera ports: added RST, SCL, SDA, TIM, {DCMI}; removed none
- sheet Display ports: added LIGHT_PWM, RST, TEAR, {FMC_LCD}; removed none
- sheet EEPROM ports: added SCL, SDA; removed none
- sheet MCU ports: added CAM_RST, CAM_TIM, I2C4_SCL, I2C4_SDA, LCD_RST, LIGHT_PWM, PWR_STATUS, SAI_FS, SAI_SCK, SAI_SD, SD_DET, TEAR, USB_DM, USB_DP, {DCMI}, {FMC_LCD}, {SD}; removed none
- sheet Microphones ports: added SAI_FS, SAI_SCK, SAI_SD, SCL, SDA, SHDNZ; removed none

Commit message: almost finished power
Other:
- sheet User interface ports: added BUTTON, DOWN, LEFT, RIGHT, TRIGGER, UP; removed none
Changed lines of the file:
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@@
 	)
 	(sheet
-		(at 132.715 123.19)
-		(size 18.415 10.795)
+		(at 189.23 119.38)
+		(size 17.78 17.78)
 		(exclude_from_sim no)
 		(in_bom yes)
@@
 		)
 		(property "Sheetname" "User interface"
-			(at 132.715 122.4784 0)
+			(at 189.23 118.6684 0)
 			(show_name no)
 			(do_not_autoplace no)
@@
 		)
 		(property "Sheetfile" "trigger.kicad_sch"
-			(at 132.715 134.5696 0)
-			(show_name no)
-			(do_not_autoplace no)
-			(effects
-				(font
-					(size 1.27 1.27)
-				)
-				(justify left top)
+			(at 189.23 137.7446 0)
+			(show_name no)
+			(do_not_autoplace no)
+			(effects
+				(font
+					(size 1.27 1.27)
+				)
+				(justify left top)
+			)
+		)
+		(pin "BUTTON" output
+			(at 189.23 121.92 180)
+			(effects
+				(font
+					(size 1.27 1.27)
+				)
+				(justify left)
+			)
+		)
+		(pin "DOWN" output
+			(at 189.23 127 180)
+			(effects
+				(font
+					(size 1.27 1.27)
+				)
+				(justify left)
+			)
+		)
+		(pin "LEFT" output
+			(at 189.23 129.54 180)
+			(effects
+				(font
+					(size 1.27 1.27)
+				)
+				(justify left)
+			)
+		)
+		(pin "RIGHT" output
+			(at 189.23 132.08 180)
+			(effects
+				(font
+					(size 1.27 1.27)
+				)
+				(justify left)
+			)
+		)
+		(pin "TRIGGER" output
+			(at 189.23 134.62 180)
+			(effects
+				(font
+					(size 1.27 1.27)
+				)
+				(justify left)
+			)
+		)
+		(pin "UP" output
+			(at 189.23 124.46 180)
+			(effects
+				(font
+					(size 1.27 1.27)
+				)
+				(justify left)
 			)
 		)
@@
 	(sheet
 		(at 102.87 43.18)
-		(size 71.12 69.215)
+		(size 71.12 93.98)
 		(exclude_from_sim no)
 		(in_bom yes)
@@
 		)
 		(property "Sheetfile" "MCU.kicad_sch"
-			(at 102.87 112.9796 0)
-			(show_name no)
-			(do_not_autoplace no)
+			(at 102.87 137.7446 0)
+			(show_name no)
+			(do_not_autoplace no)

Commit message: PCB routed
Parts:
- added H1, H2, H3, H4: M3 mounting hole, MountingHole:MountingHole_3.2mm_M3_DIN965_Pad, symbol Mechanical:MountingHole_Pad
Connections:
- new net GND: H1.1, H2.1, H3.1, H4.1
Other:
- sheet MCU ports: added BUTTON, DOWN, LEFT, RIGHT, SHDNZ, TRIGGER, UP; removed none
