File: Microphone board/SD.kicad_sch (KiCad schematic)
At the start: 9 parts, among them J1 TF-01A, U5 TPD6F003

Commit message: almost finished power
Parts:
- renumbered J1 to J3, R40 to R42, R39 to R43, R38 to R44, R37 to R45, R35 to R46, R36 to R47
Changed lines of the file:
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@@
 		(dnp no)
 		(fields_autoplaced yes)
-		(property "Reference" "R37"
+		(property "Reference" "R45"
 			(at 144.78 54.6099 0)
 			(show_name no)
@@
 			(project "Microphone board"
 				(path "/54b36551-a175-45db-a91c-236f7d72a35b/5faa6c77-3ace-4c5c-af94-e4673e5e050e"
-					(reference "R37")
+					(reference "R45")
 					(unit 1)
 				)
@@
 		(dnp no)
 		(fields_autoplaced yes)
-		(property "Reference" "R39"
+		(property "Reference" "R43"
 			(at 127 54.6099 0)
 			(show_name no)
@@
 			(project "Microphone board"
 				(path "/54b36551-a175-45db-a91c-236f7d72a35b/5faa6c77-3ace-4c5c-af94-e4673e5e050e"
-					(reference "R39")
+					(reference "R43")
 					(unit 1)
 				)
@@
 		(dnp no)
 		(fields_autoplaced yes)
-		(property "Reference" "#PWR091"
+		(property "Reference" "#PWR0105"
 			(at 81.28 91.44 0)
 			(hide yes)
@@
 			(project "Microphone board"
 				(path "/54b36551-a175-45db-a91c-236f7d72a35b/5faa6c77-3ace-4c5c-af94-e4673e5e050e"
-					(reference "#PWR091")
+					(reference "#PWR0105")
 					(unit 1)
 				)
@@
 		(dnp no)
 		(fields_autoplaced yes)
-		(property "Reference" "#PWR090"
+		(property "Reference" "#PWR0109"
 			(at 208.28 93.98 0)
 			(hide yes)
@@
 			(project "Microphone board"
 				(path "/54b36551-a175-45db-a91c-236f7d72a35b/5faa6c77-3ace-4c5c-af94-e4673e5e050e"
-					(reference "#PWR090")
+					(reference "#PWR0109")
 					(unit 1)
 				)
@@
 		(dnp no)
 		(fields_autoplaced yes)
-		(property "Reference" "J1"
+		(property "Reference" "J3"
 			(at 186.055 50.8 0)
 			(show_name no)
@@
 			(project "Microphone board"
 				(path "/54b36551-a175-45db-a91c-236f7d72a35b/5faa6c77-3ace-4c5c-af94-e4673e5e050e"
-					(reference "J1")
+					(reference "J3")
 					(unit 1)
 				)
@@
 		(dnp no)
 		(fields_autoplaced yes)
-		(property "Reference" "R40"
+		(property "Reference" "R42"
 			(at 118.11 54.6099 0)
 			(show_name no)
@@
 			(project "Microphone board"
 				(path "/54b36551-a175-45db-a91c-236f7d72a35b/5faa6c77-3ace-4c5c-af94-e4673e5e050e"
-					(reference "R40")
+					(reference "R42")
 					(unit 1)
 				)
@@
 		(dnp no)
 		(fields_autoplaced yes)
-		(property "Reference" "R38"
+		(property "Reference" "R44"
 			(at 135.89 54.6099 0)
 			(show_name no)
@@
 			(project "Microphone board"
 				(path "/54b36551-a175-45db-a91c-236f7d72a35b/5faa6c77-3ace-4c5c-af94-e4673e5e050e"
-					(reference "R38")
+					(reference "R44")
 					(unit 1)
 				)
@@
 		(dnp no)
 		(fields_autoplaced yes)
-		(property "Reference" "#PWR088"
+		(property "Reference" "#PWR0107"
 			(at 160.02 50.8 0)
 			(hide yes)
@@
 			(project "Microphone board"
 				(path "/54b36551-a175-45db-a91c-236f7d72a35b/5faa6c77-3ace-4c5c-af94-e4673e5e050e"
-					(reference "#PWR088")
+					(reference "#PWR0107")
 					(unit 1)
 				)
@@
 		(dnp no)
 		(fields_autoplaced yes)
-		(property "Reference" "#PWR089"
+		(property "Reference" "#PWR0108"
 			(at 160.02 93.98 0)
 			(hide yes)
@@
 			(project "Microphone board"
 				(path "/54b36551-a175-45db-a91c-236f7d72a35b/5faa6c77-3ace-4c5c-af94-e4673e5e050e"
-					(reference "#PWR089")
+					(reference "#PWR0108")
 					(unit 1)
 				)
@@
 		(dnp no)
 		(fields_autoplaced yes)
-		(property "Reference" "#PWR087"
+		(property "Reference" "#PWR0106"
 			(at 147.32 88.9 0)
 			(hide yes)
@@
 			(project "Microphone board"
 				(path "/54b36551-a175-45db-a91c-236f7d72a35b/5faa6c77-3ace-4c5c-af94-e4673e5e050e"
-					(reference "#PWR087")
+					(reference "#PWR0106")
 					(unit 1)
 				)
@@
 		(dnp no)
 		(fields_autoplaced yes)
-		(property "Reference" "R36"
+		(property "Reference" "R47"
 			(at 153.67 54.6099 0)
 			(show_name no)
@@
 			(project "Microphone board"
 				(path "/54b36551-a175-45db-a91c-236f7d72a35b/5faa6c77-3ace-4c5c-af94-e4673e5e050e"
-					(reference "R36")
+					(reference "R47")
 					(unit 1)
 				)
@@
 		(dnp no)
 		(fields_autoplaced yes)
-		(property "Reference" "R35"
+		(property "Reference" "R46"
 			(at 149.86 90.1699 0)
 			(show_name no)
@@
 			(project "Microphone board"
 				(path "/54b36551-a175-45db-a91c-236f7d72a35b/5faa6c77-3ace-4c5c-af94-e4673e5e050e"
-					(reference "R35")
-					(unit 1)
-				)
+					(reference "R46")
+					(unit 1)
+				)

Commit message: PCB routed
Parts:
- added C88: 100n, Capacitor_SMD:C_0402_1005Metric, symbol Device:C
Connections:
- net +3V3: now also C88.1
- net GND: now also C88.2
- net SD_D0: no longer U5.1 (Ch1_In)
- net SD_D3F: now reaches J3.2 (DAT3/CD), R45.2, U5.11 (Ch2_Out)
- net SD_CMDF: now reaches J3.3 (CMD), R44.2, U5.10 (Ch3_Out)
- net SD_D2F: now reaches J3.1 (DAT2), R47.2, U5.12 (Ch1_Out)
- net SD_D1F: now reaches J3.8 (DAT1), R41.2, U5.7 (Ch6_Out)
- net SD_D0F: now reaches J3.7 (DAT0), R42.2, U5.8 (Ch5_Out)
- net SD_CLKF: now reaches J3.5 (CLK), R43.2, U5.9 (Ch4_Out)
- new net SD_D2: U5.1 (Ch1_In)
Other:
- moved on the sheet: J3, R41, R42, R43, R44, R45, R46, R47
