File: Microphone board/usb.kicad_sch (KiCad schematic)
At the start: 6 parts, among them J4 TYPE-C 16PIN 2MD(073), U6 USBLC6-2SC6

Commit message: almost finished power
Parts:
- R56: renamed from R43; footprint (none) -> Resistor_SMD:R_01005_0402Metric
- R57: renamed from R49; footprint (none) -> Resistor_SMD:R_01005_0402Metric
- R58: renamed from R50; footprint (none) -> Resistor_SMD:R_01005_0402Metric
- R59: renamed from R51; footprint (none) -> Resistor_SMD:R_01005_0402Metric
- renumbered U6 to U11
Changed lines of the file:
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@@
 		(in_pos_files yes)
 		(dnp no)
-		(property "Reference" "R50"
+		(property "Reference" "R58"
 			(at 126.238 94.234 90)
 			(show_name no)
@@
 			)
 		)
-		(property "Footprint" ""
+		(property "Footprint" "Resistor_SMD:R_01005_0402Metric"
 			(at 130.81 97.028 90)
 			(hide yes)
@@
 			(project "Microphone board"
 				(path "/54b36551-a175-45db-a91c-236f7d72a35b/4a07b22c-fbc7-448a-93f8-173b71156924"
-					(reference "R50")
+					(reference "R58")
 					(unit 1)
 				)
@@
 		(dnp no)
 		(fields_autoplaced yes)
-		(property "Reference" "#PWR0113"
+		(property "Reference" "#PWR0135"
 			(at 146.05 81.28 0)
 			(hide yes)
@@
 			(project "Microphone board"
 				(path "/54b36551-a175-45db-a91c-236f7d72a35b/4a07b22c-fbc7-448a-93f8-173b71156924"
-					(reference "#PWR0113")
+					(reference "#PWR0135")
 					(unit 1)
 				)
@@
 		(in_pos_files yes)
 		(dnp no)
-		(property "Reference" "R51"
+		(property "Reference" "R59"
 			(at 126.238 96.774 90)
 			(show_name no)
@@
 			)
 		)
-		(property "Footprint" ""
+		(property "Footprint" "Resistor_SMD:R_01005_0402Metric"
 			(at 130.81 99.568 90)
 			(hide yes)
@@
 			(project "Microphone board"
 				(path "/54b36551-a175-45db-a91c-236f7d72a35b/4a07b22c-fbc7-448a-93f8-173b71156924"
-					(reference "R51")
+					(reference "R59")
 					(unit 1)
 				)
@@
 		(in_pos_files yes)
 		(dnp no)
-		(property "Reference" "R49"
+		(property "Reference" "R57"
 			(at 122.428 86.614 90)
 			(show_name no)
@@
 			)
 		)
-		(property "Footprint" ""
+		(property "Footprint" "Resistor_SMD:R_01005_0402Metric"
 			(at 127 89.408 90)
 			(hide yes)
@@
 			(project "Microphone board"
 				(path "/54b36551-a175-45db-a91c-236f7d72a35b/4a07b22c-fbc7-448a-93f8-173b71156924"
-					(reference "R49")
+					(reference "R57")
 					(unit 1)
 				)
@@
 		(in_pos_files yes)
 		(dnp no)
-		(property "Reference" "R43"
+		(property "Reference" "R56"
 			(at 122.428 84.074 90)
 			(show_name no)
@@
 			)
 		)
-		(property "Footprint" ""
+		(property "Footprint" "Resistor_SMD:R_01005_0402Metric"
 			(at 127 86.868 90)
 			(hide yes)
@@
 			(project "Microphone board"
 				(path "/54b36551-a175-45db-a91c-236f7d72a35b/4a07b22c-fbc7-448a-93f8-173b71156924"
-					(reference "R43")
+					(reference "R56")
 					(unit 1)
 				)
@@
 		(dnp no)
 		(fields_autoplaced yes)
-		(property "Reference" "U6"
+		(property "Reference" "U11"
 			(at 147.7011 87.63 0)
 			(show_name no)
@@
 			(project "Microphone board"
 				(path "/54b36551-a175-45db-a91c-236f7d72a35b/4a07b22c-fbc7-448a-93f8-173b71156924"
-					(reference "U6")
+					(reference "U11")
 					(unit 1)
 				)
@@
 		(dnp no)
 		(fields_autoplaced yes)
-		(property "Reference" "#PWR0110"
+		(property "Reference" "#PWR0134"
 			(at 138.43 92.71 0)
 			(hide yes)
@@
 			(project "Microphone board"
 				(path "/54b36551-a175-45db-a91c-236f7d72a35b/4a07b22c-fbc7-448a-93f8-173b71156924"
-					(reference "#PWR0110")
+					(reference "#PWR0134")
 					(unit 1)
 				)
@@
 		(dnp no)
 		(fields_autoplaced yes)
-		(property "Reference" "#PWR0112"
+		(property "Reference" "#PWR0136"
 			(at 146.05 111.76 0)
 			(hide yes)
@@
 			(project "Microphone board"
 				(path "/54b36551-a175-45db-a91c-236f7d72a35b/4a07b22c-fbc7-448a-93f8-173b71156924"
-					(reference "#PWR0112")
+					(reference "#PWR0136")
 					(unit 1)
 				)
@@
 		(dnp no)
 		(fields_autoplaced yes)
-		(property "Reference" "#PWR0111"
+		(property "Reference" "#PWR0133"
 			(at 105.41 129.54 0)
 			(hide yes)
@@
 			(project "Microphone board"
 				(path "/54b36551-a175-45db-a91c-236f7d72a35b/4a07b22c-fbc7-448a-93f8-173b71156924"
-					(reference "#PWR0111")
-					(unit 1)
-				)
+					(reference "#PWR0133")
+					(unit 1)
+				)

Commit message: PCB routed
Parts:
- R56, R57, R58, R59: footprint Resistor_SMD:R_01005_0402Metric -> Resistor_SMD:R_0402_1005Metric
Connections:
- net USB_IN_N: now reaches J4.A7 (D-), J4.B7 (D-), R58.1
- net USB_U_N: now reaches R58.2, U11.1 (I/O1)
- net USB_IN_P: now reaches J4.A6 (D+), J4.B6 (D+), R59.1
- net USB_U_P: now reaches R59.2, U11.3 (I/O2)
Other:
- moved on the sheet: R56, R57, R58, R59, U11
