File: Microphone board/microphones.kicad_sch (KiCad schematic)
At the start: 0 parts

Commit message: Made almost the rest of the schematic lol
Parts:
- added C10, C11, C12, C13, C14, C15, C16, C17, C18, C19, C20, C21, C22, C23, C24, C9: 100n, Capacitor_SMD:C_0402_1005Metric, symbol Device:C_Small
- added C2, C3, C5, C7: 2.2u, Capacitor_SMD:C_0402_1005Metric, symbol Device:C
- added C25, C26, C27, C4, C6, C8: 100n, Capacitor_SMD:C_0402_1005Metric, symbol Device:C
- added M1, M10, M11, M12, M13, M14, M15, M16, M2, M3, M4, M5, M6, M7, M8, M9: MSM261DDB019, Mic_Parts:MSM261DDB019, symbol Mic_Parts:MSM261DDB019
- added R10, R11, R12, R13, R14, R15, R16, R17, R18, R19, R20, R21, R22, R23, R24, R25, R26, R27, R28, R29, R30, R31, R32, R33, R34, R7, R8, R9: 33R, Resistor_SMD:R_0402_1005Metric, symbol Device:R
- added R5, R6: 10k, Resistor_SMD:R_0402_1005Metric, symbol Device:R
- added U3, U4: TLV320ADC5140IRTWT, Mic_Parts:RTW24_4P15X4P15_TEX, symbol Mic_Parts:TLV320ADC5140IRTWT
Connections:
- new net: M7.1 (DAT), R19.1
- new net: M14.1 (DAT), R25.1
- new net: M3.1 (DAT), R18.1
- new net: R31.1, U3.21 (SDOUT)
- new net: C7.1, U4.24 (DREG)
- new net: R34.1, U4.21 (SDOUT)
- new net: R34.2, U3.20 (GPIO1)
- new net: M2.1 (DAT), R16.1
- new net: M8.1 (DAT), R21.1
- new net: M6.1 (DAT), R22.1
- new net: R7.2, U3.7 (IN1M_GPO1)
- new net: R12.2, U4.9 (IN2M_GPO2)
- new net: R13.2, U4.11 (IN3M_GPO3)
- new net: C4.1, U3.3 (VREF)
- new net: M1.1 (DAT), R15.1
- new net: R32.1, U3.23 (FSYNC)
- new net: M15.1 (DAT), R27.1
- new net: M11.1 (DAT), R28.1
- new net: R33.1, U3.22 (BCLK)
- new net: R11.2, U4.7 (IN1M_GPO1)
- new net: M16.1 (DAT), R29.1
- new net: C3.1, U4.2 (AREG)
- new net: M5.1 (DAT), R20.1
- new net: R9.2, U3.11 (IN3M_GPO3)
- new net: R10.2, U3.13 (IN4M_GPO4)
- new net: R8.2, U3.9 (IN2M_GPO2)
- new net: M12.1 (DAT), R30.1
- new net: M9.1 (DAT), R24.1
- new net: R14.2, U4.13 (IN4M_GPO4)
- new net: M13.1 (DAT), R23.1
- new net: M4.1 (DAT), R17.1
- new net: M10.1 (DAT), R26.1
- new net: C6.1, U4.3 (VREF)
- new net: C2.1, U3.2 (AREG)
- new net: C5.1, U3.24 (DREG)
- new net +3V3: C25.1, C26.1, R5.1, R6.1, U3.19 (IOVDD), U4.16 (ADDR0_SCLK), U4.19 (IOVDD)
- new net +3V3A: C10.1, C11.1, C12.1, C13.1, C14.1, C15.1, C16.1, C17.1, C18.1, C19.1, C20.1, C21.1, C22.1, C23.1, C24.1, C27.1, C8.1, C9.1, M1.2 (SEL), M1.5 (VDD), M10.5 (VDD), M11.5 (VDD), M12.5 (VDD), M13.2 (SEL), M13.5 (VDD), M14.2 (SEL), M14.5 (VDD), M15.2 (SEL), M15.5 (VDD), M16.2 (SEL), M16.5 (VDD), M2.5 (VDD), M3.5 (VDD), M4.2 (SEL), M4.5 (VDD), M5.5 (VDD), M6.5 (VDD), M7.2 (SEL), M7.5 (VDD), M8.2 (SEL), M8.5 (VDD), M9.5 (VDD), U3.1 (AVDD), U4.1 (AVDD)
- new net CH1_CLK: M1.4 (CLK), M2.4 (CLK), R7.1
- new net CH1_DAT: R15.2, R16.2, U3.6 (IN1P_GPI1)
- new net CH2_CLK: M3.4 (CLK), M4.4 (CLK), R8.1
- new net CH2_DAT: R17.2, R18.2, U3.8 (IN2P_GPI2)
- new net CH3_CLK: M5.4 (CLK), M7.4 (CLK), R9.1
- new net CH3_DAT: R19.2, R20.2, U3.10 (IN3P_GPI3)
- new net CH4_CLK: M6.4 (CLK), M8.4 (CLK), R10.1
- new net CH4_DAT: R21.2, R23.2, U3.12 (IN4P_GPI4)
- new net CH5_CLK: M14.4 (CLK), M9.4 (CLK), R11.1
- new net CH5_DAT: R24.2, R25.2, U4.6 (IN1P_GPI1)
- new net CH6_CLK: M10.4 (CLK), M15.4 (CLK), R12.1
- new net CH6_DAT: R26.2, R27.2, U4.8 (IN2P_GPI2)
- new net CH7_CLK: M11.4 (CLK), R13.1
- new net CH7_DAT: R28.2, U4.10 (IN3P_GPI3)
- new net CH8_CLK: M12.4 (CLK), M16.4 (CLK), R14.1
- new net CH8_DAT: R29.2, R30.2, U4.12 (IN4P_GPI4)
- new net GND: C10.2, C11.2, C12.2, C13.2, C14.2, C15.2, C16.2, C17.2, C18.2, C19.2, C2.2, C20.2, C21.2, C22.2, C23.2, C24.2, C25.2, C26.2, C27.2, C3.2, C4.2, C5.2, C6.2, C7.2, C8.2, C9.2, M1.3 (GND), M10.2 (SEL), M10.3 (GND), M11.2 (SEL), M11.3 (GND), M12.2 (SEL), M12.3 (GND), M13.3 (GND), M14.3 (GND), M15.3 (GND), M16.3 (GND), M2.2 (SEL), M2.3 (GND), M3.2 (SEL), M3.3 (GND), M4.3 (GND), M5.2 (SEL), M5.3 (GND), M6.2 (SEL), M6.3 (GND), M7.3 (GND), M8.3 (GND), M9.2 (SEL), M9.3 (GND), U3.15 (ADDR1_MISO), U3.16 (ADDR0_SCLK), U3.25 (EPAD), U3.4 (AVSS), U4.15 (ADDR1_MISO), U4.25 (EPAD), U4.4 (AVSS)
- new net SAI_FS: R32.2, U4.23 (FSYNC)
- new net SAI_SCK: R33.2, U4.22 (BCLK)
- new net SAI_SD: R31.2
- new net SCL: U3.17 (SCL_MOSI), U4.17 (SCL_MOSI)
- new net SDA: U3.18 (SDA_SSZ), U4.18 (SDA_SSZ)
- new net SHDNZ: R5.2, R6.2, U3.14 (SHDNZ), U4.14 (SHDNZ)
- no-connect marks 0 -> 3
Other:
- note added: "I2C"
- note added: "Place all 33R near source"
- note added: "SAI"
- note added: "all these should be 50Z"
- note added: "configure GPIO_CFG[3:0] to 11d also configure this one as master"

Commit message: almost finished power
Parts:
- removed R13, R25, R26, R27, R28, R29, R30: 33R, Resistor_SMD:R_0402_1005Metric, symbol Device:R
- added R10, R15, R5, R6, R7, R8, R9: 22R, Resistor_SMD:R_0402_1005Metric, symbol Device:R
- R11, R12, R14, R16, R17, R18, R19, R20, R21, R22, R23, R24: value 33R -> 22R
- R13: renamed from R15; value 33R -> 22R
- renumbered C10 to C41, C11 to C42, C13 to C43, C14 to C44, C17 to C45, C18 to C46, C19 to C47, C20 to C48, C9 to C49, C12 to C50, C15 to C51, C16 to C52, C21 to C53, C22 to C54, C23 to C55, C24 to C56, C2 to C57, C3 to C58, C4 to C59, C6 to C60, C5 to C61, C7 to C62, C25 to C63, C26 to C64, C8 to C65, C27 to C66, M2 to M1, M4 to M10, M7 to M11, M8 to M12, M3 to M2, M5 to M3, M6 to M4, M9 to M5, M10 to M6, M11 to M7, M12 to M8, M1 to M9, R7 to R25, R8 to R26, R9 to R27, R10 to R28, R34 to R29, R31 to R30, R32 to R31, R33 to R32, R5 to R33, R6 to R34
Connections:
- net CH1_DAT: now also R5.2; no longer R16.2
- net CH2_DAT: now also R14.2, R6.2; no longer R17.2, R18.2
- net CH3_DAT: now also R15.2, R7.2; no longer R19.2, R20.2
- net CH4_DAT: now also R16.2, R8.2; no longer R21.2, R23.2
- net CH5_CLK: now also M13.4 (CLK), R21.1; no longer M14.4 (CLK), R11.1
- net CH5_DAT: now also R17.2, R9.2; no longer R24.2
- net CH6_CLK: now also M14.4 (CLK), R22.1; no longer M15.4 (CLK), R12.1
- net CH6_DAT: now also R18.2, R10.2
- net CH7_CLK: now also M15.4 (CLK), R23.1
- net CH7_DAT: now also R11.2, R19.2
- net CH8_CLK: now also R24.1; no longer R14.1
- net CH8_DAT: now also R12.2, R20.2
- net at M11.1 (DAT): now also R15.1; no longer R19.1
- net at M14.1 (DAT): now also R18.1
- net at M2.1 (DAT): now also R6.1; no longer R18.1
- net at M1.1 (DAT): now also R5.1; no longer R16.1
- net at M12.1 (DAT): now also R16.1; no longer R21.1
- net at M4.1 (DAT): now also R8.1; no longer R22.1
- net at R22.2: now also U4.9 (IN2M_GPO2)
- net at U4.11 (IN3M_GPO3): now also R23.2
- net at M15.1 (DAT): now also R19.1
- net at M7.1 (DAT): now also R11.1
- net at U4.7 (IN1M_GPO1): now also R21.2; no longer R11.2
- net at M16.1 (DAT): now also R20.1
- net at M3.1 (DAT): now also R7.1; no longer R20.1
- net at M8.1 (DAT): now also R12.1
- net at M5.1 (DAT): now also R9.1; no longer R24.1
- net at U4.13 (IN4M_GPO4): now also R24.2; no longer R14.2
- net at M13.1 (DAT): now also R17.1; no longer R23.1
- net at M10.1 (DAT): now also R14.1; no longer R17.1
- net at M6.1 (DAT): now also R10.1

Commit message: PCB routed
Parts:
- R29, R30, R31, R32: value 33R -> 22R
- renumbered M9 to M1, M5 to M10, M14 to M11, M6 to M12, M15 to M13, M7 to M14, M16 to M15, M8 to M16, M1 to M2, M10 to M3, M2 to M4, M11 to M5, M3 to M6, M12 to M7, M4 to M8, M13 to M9
Changed lines of the file:
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@@
 		(dnp no)
 		(fields_autoplaced yes)
-		(property "Reference" "M14"
+		(property "Reference" "M11"
 			(at 114.3 168.91 0)
 			(show_name no)
@@
 			(project "Microphone board"
 				(path "/54b36551-a175-45db-a91c-236f7d72a35b/46472c5b-0bf6-4ffe-840a-aba929ed84f5"
-					(reference "M14")
+					(reference "M11")
 					(unit 1)
 				)
@@
 		(dnp no)
 		(fields_autoplaced yes)
-		(property "Reference" "M2"
+		(property "Reference" "M4"
 			(at 86.36 72.39 0)
 			(show_name no)
@@
 			(project "Microphone board"
 				(path "/54b36551-a175-45db-a91c-236f7d72a35b/46472c5b-0bf6-4ffe-840a-aba929ed84f5"
-					(reference "M2")
+					(reference "M4")
 					(unit 1)
 				)
@@
 			)
 		)
-		(property "Value" "33R"
+		(property "Value" "22R"
 			(at 220.472 67.564 90)
 			(show_name no)
@@
 			)
 		)
-		(property "Value" "33R"
+		(property "Value" "22R"
 			(at 213.36 175.26 90)
 			(show_name no)
@@
 		(dnp no)
 		(fields_autoplaced yes)
-		(property "Reference" "M4"
+		(property "Reference" "M8"
 			(at 86.36 128.27 0)
 			(show_name no)
@@
 			(project "Microphone board"
 				(path "/54b36551-a175-45db-a91c-236f7d72a35b/46472c5b-0bf6-4ffe-840a-aba929ed84f5"
-					(reference "M4")
+					(reference "M8")
 					(unit 1)
 				)
@@
 			)
 		)
-		(property "Value" "33R"
+		(property "Value" "22R"
 			(at 220.472 70.104 90)
 			(show_name no)
@@
 			)
 		)
-		(property "Value" "33R"
+		(property "Value" "22R"
 			(at 220.472 72.644 90)
 			(show_name no)
@@
 		(dnp no)
 		(fields_autoplaced yes)
-		(property "Reference" "M16"
+		(property "Reference" "M15"
 			(at 114.3 224.79 0)
 			(show_name no)
@@
 			(project "Microphone board"
 				(path "/54b36551-a175-45db-a91c-236f7d72a35b/46472c5b-0bf6-4ffe-840a-aba929ed84f5"
-					(reference "M16")
+					(reference "M15")
 					(unit 1)
 				)
@@
 		(dnp no)
 		(fields_autoplaced yes)
-		(property "Reference" "M11"
+		(property "Reference" "M5"
 			(at 114.3 85.09 0)
 			(show_name no)
@@
 			(project "Microphone board"
 				(path "/54b36551-a175-45db-a91c-236f7d72a35b/46472c5b-0bf6-4ffe-840a-aba929ed84f5"
-					(reference "M11")
+					(reference "M5")
 					(unit 1)
 				)
@@
 		(dnp no)
 		(fields_autoplaced yes)
-		(property "Reference" "M12"
+		(property "Reference" "M7"
 			(at 114.3 113.03 0)
 			(show_name no)
@@
 			(project "Microphone board"
 				(path "/54b36551-a175-45db-a91c-236f7d72a35b/46472c5b-0bf6-4ffe-840a-aba929ed84f5"
-					(reference "M12")
+					(reference "M7")
 					(unit 1)
 				)
@@
 		(dnp no)
 		(fields_autoplaced yes)
-		(property "Reference" "M7"
+		(property "Reference" "M14"
 			(at 86.36 212.09 0)
 			(show_name no)
@@
 			(project "Microphone board"
 				(path "/54b36551-a175-45db-a91c-236f7d72a35b/46472c5b-0bf6-4ffe-840a-aba929ed84f5"
-					(reference "M7")
+					(reference "M14")
 					(unit 1)
 				)
@@
 		(dnp no)
 		(fields_autoplaced yes)
-		(property "Reference" "M1"
+		(property "Reference" "M2"
 			(at 86.36 44.45 0)
 			(show_name no)
@@
 			(project "Microphone board"
 				(path "/54b36551-a175-45db-a91c-236f7d72a35b/46472c5b-0bf6-4ffe-840a-aba929ed84f5"
-					(reference "M1")
+					(reference "M2")
 					(unit 1)
 				)
@@
 		(dnp no)
 		(fields_autoplaced yes)
-		(property "Reference" "M9"
+		(property "Reference" "M1"
 			(at 114.3 29.21 0)
 			(show_name no)
@@
 			(project "Microphone board"
 				(path "/54b36551-a175-45db-a91c-236f7d72a35b/46472c5b-0bf6-4ffe-840a-aba929ed84f5"
-					(reference "M9")
+					(reference "M1")
 					(unit 1)
 				)
@@
 		(dnp no)
 		(fields_autoplaced yes)
-		(property "Reference" "M13"
+		(property "Reference" "M9"
 			(at 114.3 140.97 0)
 			(show_name no)
@@
 			(project "Microphone board"
 				(path "/54b36551-a175-45db-a91c-236f7d72a35b/46472c5b-0bf6-4ffe-840a-aba929ed84f5"
-					(reference "M13")
+					(reference "M9")
 					(unit 1)
 				)
@@
 		(dnp no)
 		(fields_autoplaced yes)
-		(property "Reference" "M15"
+		(property "Reference" "M13"
 			(at 114.3 196.85 0)
 			(show_name no)
@@
 			(project "Microphone board"
 				(path "/54b36551-a175-45db-a91c-236f7d72a35b/46472c5b-0bf6-4ffe-840a-aba929ed84f5"
-					(reference "M15")
+					(reference "M13")
 					(unit 1)
 				)
@@
 		(dnp no)
 		(fields_autoplaced yes)
-		(property "Reference" "M10"
+		(property "Reference" "M3"
 			(at 114.3 57.15 0)
 			(show_name no)
@@
 			(project "Microphone board"
 				(path "/54b36551-a175-45db-a91c-236f7d72a35b/46472c5b-0bf6-4ffe-840a-aba929ed84f5"
-					(reference "M10")
+					(reference "M3")
 					(unit 1)
 				)
@@
 		(dnp no)
 		(fields_autoplaced yes)
-		(property "Reference" "M5"
+		(property "Reference" "M10"
 			(at 86.36 156.21 0)
 			(show_name no)
@@
 			(project "Microphone board"
 				(path "/54b36551-a175-45db-a91c-236f7d72a35b/46472c5b-0bf6-4ffe-840a-aba929ed84f5"
-					(reference "M5")
+					(reference "M10")
 					(unit 1)
 				)
@@
 		(dnp no)
 		(fields_autoplaced yes)
-		(property "Reference" "M6"
+		(property "Reference" "M12"
 			(at 86.36 184.15 0)
 			(show_name no)
@@
 			(project "Microphone board"
 				(path "/54b36551-a175-45db-a91c-236f7d72a35b/46472c5b-0bf6-4ffe-840a-aba929ed84f5"
-					(reference "M6")
+					(reference "M12")
 					(unit 1)
 				)
@@
 		(dnp no)
 		(fields_autoplaced yes)
-		(property "Reference" "M3"
+		(property "Reference" "M6"
 			(at 86.36 100.33 0)
 			(show_name no)
@@
 			(project "Microphone board"
 				(path "/54b36551-a175-45db-a91c-236f7d72a35b/46472c5b-0bf6-4ffe-840a-aba929ed84f5"
-					(reference "M3")
+					(reference "M6")
 					(unit 1)
 				)
@@
 		(dnp no)
 		(fields_autoplaced yes)
-		(property "Reference" "M8"
+		(property "Reference" "M16"
 			(at 86.36 240.03 0)
 			(show_name no)
@@
 			(project "Microphone board"
 				(path "/54b36551-a175-45db-a91c-236f7d72a35b/46472c5b-0bf6-4ffe-840a-aba929ed84f5"
-					(reference "M8")
+					(reference "M16")
 					(unit 1)
 				)

Commit message: finished r1 of the board
Parts:
- R25, R26, R27, R28: value 33R -> 22R
Changed lines of the file:
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@@
 		(dnp no)
 		(property "Reference" "R25"
-			(at 163.83 72.644 90)
+			(at 163.068 72.644 90)
 			(show_name no)
 			(do_not_autoplace no)
@@
 			)
 		)
-		(property "Value" "33R"
+		(property "Value" "22R"
 			(at 172.212 72.644 90)
 			(show_name no)
@@
 		(dnp no)
 		(property "Reference" "R27"
-			(at 163.83 82.804 90)
+			(at 163.068 82.804 90)
 			(show_name no)
 			(do_not_autoplace no)
@@
 			)
 		)
-		(property "Value" "33R"
+		(property "Value" "22R"
 			(at 172.212 82.804 90)
 			(show_name no)
@@
 			)
 		)
-		(property "Value" "33R"
+		(property "Value" "22R"
 			(at 172.212 87.884 90)
 			(show_name no)
@@
 		(dnp no)
 		(property "Reference" "R26"
-			(at 163.83 77.724 90)
+			(at 163.068 77.724 90)
 			(show_name no)
 			(do_not_autoplace no)
@@
 			)
 		)
-		(property "Value" "33R"
+		(property "Value" "22R"
 			(at 172.212 77.724 90)
 			(show_name no)
