File: Microphone board/microphones.kicad_sch (KiCad schematic)
At the start: 74 parts, among them M1 MSM261DDB019, M10 MSM261DDB019, M11 MSM261DDB019, M12 MSM261DDB019, M13 MSM261DDB019, M14 MSM261DDB019, M15 MSM261DDB019, M16 MSM261DDB019, M2 MSM261DDB019, M3 MSM261DDB019, M4 MSM261DDB019, M5 MSM261DDB019, M6 MSM261DDB019, M7 MSM261DDB019, M8 MSM261DDB019, M9 MSM261DDB019, U3 TLV320ADC5140IRTWT, U4 TLV320ADC5140IRTWT

Commit message: Syncing stuff between computers
Parts:
- removed R31, R32: 22R, Resistor_SMD:R_0402_1005Metric, symbol Device:R
Connections:
- net SAI_FS: now also U3.23 (FSYNC)
- net SAI_SCK: now also U3.22 (BCLK)
Changed lines of the file:
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@@
 	(wire
 		(pts
-			(xy 219.71 73.66) (xy 232.41 73.66)
-		)
-		(stroke
-			(width 0)
-			(type default)
-		)
-	)
-	(wire
-		(pts
 			(xy 102.87 124.46) (xy 105.41 124.46)
 		)
@@
 	(wire
 		(pts
-			(xy 208.28 71.12) (xy 212.09 71.12)
+			(xy 208.28 71.12) (xy 232.41 71.12)
 		)
 		(stroke
@@
 	(wire
 		(pts
-			(xy 219.71 71.12) (xy 232.41 71.12)
-		)
-		(stroke
-			(width 0)
-			(type default)
-		)
-	)
-	(wire
-		(pts
 			(xy 74.93 251.46) (xy 74.93 254)
 		)
@@
 	(wire
 		(pts
-			(xy 208.28 73.66) (xy 212.09 73.66)
+			(xy 208.28 73.66) (xy 232.41 73.66)
 		)
 		(stroke
@@
 	(symbol
 		(lib_id "Device:R")
-		(at 215.9 71.12 90)
-		(unit 1)
-		(body_style 1)
-		(exclude_from_sim no)
-		(in_bom yes)
-		(on_board yes)
-		(in_pos_files yes)
-		(dnp no)
-		(property "Reference" "R31"
-			(at 211.328 70.104 90)
-			(show_name no)
-			(do_not_autoplace no)
-			(effects
-				(font
-					(size 1.27 1.27)
-				)
-			)
-		)
-		(property "Value" "22R"
-			(at 220.472 70.104 90)
-			(show_name no)
-			(do_not_autoplace no)
-			(effects
-				(font
-					(size 1.27 1.27)
-				)
-			)
-		)
-		(property "Footprint" "Resistor_SMD:R_0402_1005Metric"
-			(at 215.9 72.898 90)
-			(hide yes)
-			(show_name no)
-			(do_not_autoplace no)
-			(effects
-				(font
-					(size 1.27 1.27)
-				)
-			)
-		)
-		(property "Datasheet" ""
-			(at 215.9 71.12 0)
-			(hide yes)
-			(show_name no)
-			(do_not_autoplace no)
-			(effects
-				(font
-					(size 1.27 1.27)
-				)
-			)
-		)
-		(property "Description" "Resistor"
-			(at 215.9 71.12 0)
-			(hide yes)
-			(show_name no)
-			(do_not_autoplace no)
-			(effects
-				(font
-					(size 1.27 1.27)
-				)
-			)
-		)
-		(pin "1"
-		)
-		(pin "2"
-		)
-		(instances
-			(project "Microphone board"
-				(path "/54b36551-a175-45db-a91c-236f7d72a35b/46472c5b-0bf6-4ffe-840a-aba929ed84f5"
-					(reference "R31")
-					(unit 1)
-				)
-			)
-		)
-	)
-	(symbol
-		(lib_id "Device:R")
 		(at 232.41 194.31 0)
 		(unit 1)
@@
 					(unit 1)
 				)
-			)
-		)
-	)
-	(symbol
-		(lib_id "Device:R")
-		(at 215.9 73.66 90)
-		(unit 1)
-		(body_style 1)
-		(exclude_from_sim no)
-		(in_bom yes)
-		(on_board yes)
-		(in_pos_files yes)
-		(dnp no)
-		(property "Reference" "R32"
-			(at 211.328 72.644 90)
-			(show_name no)
-			(do_not_autoplace no)
-			(effects
-				(font
-					(size 1.27 1.27)
-				)
-			)
-		)
-		(property "Value" "22R"
-			(at 220.472 72.644 90)
-			(show_name no)
-			(do_not_autoplace no)
-			(effects
-				(font
-					(size 1.27 1.27)
-				)
-			)
-		)
-		(property "Footprint" "Resistor_SMD:R_0402_1005Metric"
-			(at 215.9 75.438 90)
-			(hide yes)
-			(show_name no)
-			(do_not_autoplace no)
-			(effects
-				(font
-					(size 1.27 1.27)
-				)
-			)
-		)
-		(property "Datasheet" ""
-			(at 215.9 73.66 0)
-			(hide yes)
-			(show_name no)
-			(do_not_autoplace no)
-			(effects
-				(font
-					(size 1.27 1.27)
-				)
-			)
-		)
-		(property "Description" "Resistor"
-			(at 215.9 73.66 0)
-			(hide yes)
-			(show_name no)
-			(do_not_autoplace no)
-			(effects
-				(font
-					(size 1.27 1.27)
-				)
-			)
-		)
-		(pin "1"
-		)
-		(pin "2"
-		)
-		(instances
-			(project "Microphone board"
-				(path "/54b36551-a175-45db-a91c-236f7d72a35b/46472c5b-0bf6-4ffe-840a-aba929ed84f5"
-					(reference "R32")
-					(unit 1)
-				)
