File: Microphone board/power.kicad_sch (KiCad schematic)
At the start: 22 parts, among them U10 TPS63001, U7 AP63203WU, U8 TPS7A2033PDBV, U9 TPS2116DRL

Commit message: almost finished power
Parts:
- added BT1: 3.7V 18650, Connector_Wire:SolderWire-1.5sqmm_1x02_P6mm_D1.7mm_OD3mm, symbol Device:Battery_Cell
- added C86, C87: 1u, symbol Device:C
- added D1: Green, PCM_JLCPCB:D_0603, symbol PCM_JLCPCB-Diodes:LED,0603,Yellow
- added D2: Yellow, PCM_JLCPCB:D_0603, symbol PCM_JLCPCB-Diodes:LED,0603,Yellow
- added D3: Red, PCM_JLCPCB:D_0603, symbol PCM_JLCPCB-Diodes:LED,0603,Red
- added R53, R54, R55: 470R, Resistor_SMD:R_01005_0402Metric, symbol Device:R
- added R60: 1k, Resistor_SMD:R_01005_0402Metric, symbol Device:R
- added TH1: 10k, symbol Device:Thermistor_NTC
- added U9: MCP73833-xxx-MF, Package_DFN_QFN:DFN-10-1EP_3x3mm_P0.5mm_EP1.58x2.35mm, symbol Battery_Management:MCP73833-xxx-MF
- R48: renamed from R54; footprint (none) -> Resistor_SMD:R_01005_0402Metric
- R49: renamed from R55; footprint (none) -> Resistor_SMD:R_01005_0402Metric
- R50: renamed from R56; footprint (none) -> Resistor_SMD:R_01005_0402Metric
- R51: renamed from R52; footprint (none) -> Resistor_SMD:R_01005_0402Metric
- R52: renamed from R53; footprint (none) -> Resistor_SMD:R_01005_0402Metric
- renumbered C85 to C75, C84 to C76, C81 to C77, C82 to C78, C83 to C79, C75 to C80, C76 to C81, C77 to C82, C78 to C83, C79 to C84, C80 to C85, L3 to L2, L2 to L3, U8 to U10, U10 to U6, U9 to U7, U7 to U8
Connections:
- net GND: now also BT1.2 (-), C86.2, C87.2, R60.2, TH1.2, U9.11 (EP), U9.5 (V_{SS})
- net VBAT: now also BT1.1 (+), C87.1, U9.10 (V_{BAT}), U9.9 (V_{BAT})
- net VBUS: now also C86.1, D1.2, D2.2, D3.2, U9.1 (V_{DD}), U9.2 (V_{DD})
- new net: D2.1, R54.1
- new net: D3.1, R53.1
- new net: R53.2, U9.3 (STAT1)
- new net: TH1.1, U9.8 (THERM)
- new net: R60.1, U9.6 (PROG)
- new net: R54.2, U9.4 (STAT2)
- new net: D1.1, R55.1
- new net: R55.2, U9.7 (~{PG})
Other:
- note added: "LiPo charger"
- moved on the sheet: C75, C76, C77, C78, C79, C80, C81, C82, C83, C84, C85, L2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

Commit message: PCB routed
Parts:
- C75, C78, C79, C82, C83: footprint (none) -> Capacitor_SMD:C_0805_2012Metric
- C76, C77, C81: footprint (none) -> Capacitor_SMD:C_0402_1005Metric
- C80, C84, C85, C86, C87: footprint (none) -> Capacitor_SMD:C_0603_1608Metric
- L2: value 2.2u -> GNR4018S2R2MT; footprint (none) -> Inductor_SMD:L_Abracon_ASPI-4030S
- L3: value 4.7u -> FNR5040S4R7MT; footprint (none) -> Inductor_SMD:L_Changjiang_FNR5040S
- R48, R49, R50, R51, R52, R53, R54, R55, R60: footprint Resistor_SMD:R_01005_0402Metric -> Resistor_SMD:R_0402_1005Metric
- TH1: footprint (none) -> Connector_JST:JST_PH_B2B-PH-K_1x02_P2.00mm_Vertical
Connections:
- net at C81.1, L3.1: now also U8.5 (SW); no longer U8.6 (BST)
- net at C81.2: now also U8.6 (BST); no longer U8.5 (SW)
Other:
- moved on the sheet: C75, C76, C82, C83, L2, L3, R50

Commit message: finished r1 of the board
Parts:
- added D4, D5: Red, PCM_JLCPCB:D_0603, symbol PCM_JLCPCB-Diodes:LED,0603,Red
- added R68, R69: 470R, Resistor_SMD:R_0402_1005Metric, symbol Device:R
Connections:
- net +3V3: now also R68.1
- net +5V: now also R69.1
- net GND: now also D4.1, D5.1
- new net: D4.2, R68.2
- new net: D5.2, R69.2
Other:
- note removed: "ferrite choke?"
