File: Microphone board/power.kicad_sch (KiCad schematic)
At the start: 38 parts, among them U10 TPS7A2033PDBV, U6 TPS63001, U7 TPS2116DRL, U8 AP63203WU, U9 MCP73833-xxx-MF

Commit message: Created python visualization
Other:
- note added: "Create 2.8V analog rail"
Changed lines of the file:
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@@
+		)
+	)
+	(text "Create 2.8V analog rail"
+		(exclude_from_sim no)
+		(at 179.07 155.448 0)
+		(effects
+			(font
+				(size 5.08 5.08)
+				(thickness 1.016)
+				(bold yes)
+				(color 255 0 3 1)
+			)
 		)
 	)
