File: Microphone board/MCU.kicad_sch (KiCad schematic)
At the start: 7 parts, among them U1 STM32H747XIH6, Y1 SX2M25.000M20F30TNN

Commit message: Made almost the rest of the schematic lol
Parts:
- added C28, C62: 4.7u, Capacitor_SMD:C_0603_1608Metric, symbol Device:C
- added C29: 220pF, Capacitor_SMD:C_0402_1005Metric, symbol Device:C
- added C30, C31: 10u, Capacitor_SMD:C_0805_2012Metric, symbol Device:C
- added C32, C33, C34: 2.2u, Capacitor_SMD:C_0402_1005Metric, symbol Device:C
- added C35, C36, C37, C38, C39, C40, C41, C42, C43, C44, C45, C46, C47, C48, C49, C50, C51, C52, C53, C54, C55, C56, C57, C58, C59, C60, C61, C64: 100n, Capacitor_SMD:C_0201_0603Metric, symbol Device:C
- added C63, C65: 1u, Capacitor_SMD:C_0603_1608Metric, symbol Device:C
- added L1: 2.2u, symbol Device:L
- added R3, R4: 2k2, Resistor_SMD:R_0402_1005Metric, symbol Device:R
- C1: footprint (none) -> Capacitor_SMD:C_0402_1005Metric
- R1, R2: footprint (none) -> Resistor_SMD:R_0402_1005Metric
Connections:
- net LTDC_G6 is gone; now on net SD_DET: U1.A15 (PI1)
- net +3V3: now also U1.A6 (VDDLDO), U1.B1 (VBAT), U1.C17 (VDDLDO), U1.E11 (VDD), U1.E6 (VDD), U1.E9 (VDD), U1.F17 (VDD33_USB), U1.F5 (VDD), U1.G13 (VDD), U1.G17 (VDD50_USB), U1.G2 (VFBSMPS), U1.G5 (VDD), U1.H13 (VDD), U1.H5 (VDD), U1.J13 (VDD), U1.K13 (VDD), U1.K5 (VDD), U1.L13 (VDD), U1.L5 (VDD), U1.M13 (VDD), U1.M5 (VDD), U1.N10 (VDD), U1.N11 (VDD), U1.N12 (VDD), U1.N7 (VDD), U1.N8 (VDD), U1.P17 (VDDDSI), U1.U12 (VDDLDO), C30.1, C31.1, C35.1, C36.1, C37.1, C38.1, C39.1, C40.1, C41.1, C42.1, C43.1, C44.1, C45.1, C46.1, C47.1, C48.1, C49.1, C50.1, C51.1, C52.1, C53.1, C54.1, C55.1, C56.1, C57.1, C58.1, C59.1, C60.1, C61.1, C62.1, C63.1, L1.2, R3.1, R4.1
- net GND: now also U1.A1 (VSS), U1.A17 (VSS), U1.B2 (VSS), U1.B6 (VSS), U1.C10 (VSS), U1.C13 (VSS), U1.C16 (VSS), U1.F2 (VSSSMPS), U1.G10 (VSS), U1.G11 (VSS), U1.G16 (VSS), U1.G7 (VSS), U1.G8 (VSS), U1.G9 (VSS), U1.H10 (VSS), U1.H11 (VSS), U1.H7 (VSS), U1.H8 (VSS), U1.H9 (VSS), U1.J10 (VSS), U1.J11 (VSS), U1.J16 (VSS), U1.J17 (VSS), U1.J3 (VSS), U1.J7 (VSS), U1.J8 (VSS), U1.J9 (VSS), U1.K10 (VSS), U1.K11 (VSS), U1.K15 (VSSDSI), U1.K7 (VSS), U1.K8 (VSS), U1.K9 (VSS), U1.L10 (VSS), U1.L11 (VSS), U1.L7 (VSS), U1.L8 (VSS), U1.L9 (VSS), U1.N1 (VREF-), U1.N16 (VSS), U1.P1 (VSSA), U1.R4 (VSS), U1.R8 (VSS), U1.T12 (VSS), U1.U1 (VSS), U1.U17 (VSS), C28.2, C29.2, C30.2, C31.2, C32.2, C33.2, C34.2, C35.2, C36.2, C37.2, C38.2, C39.2, C40.2, C41.2, C42.2, C43.2, C44.2, C45.2, C46.2, C47.2, C48.2, C49.2, C50.2, C51.2, C52.2, C53.2, C54.2, C55.2, C56.2, C57.2, C58.2, C59.2, C60.2, C61.2, C62.2, C63.2, C64.2, C65.2
- net SD_DET: no longer U1.A12 (PD4)
- net PWR_STATUS: now reaches U1.H17 (PK2)
- net at U1.A7 (VCAP): now also U1.D17 (VCAP), U1.U11 (VCAP), C32.1, C33.1
- net at U1.E1 (VLXSMPS): now also C29.1, L1.1
- net at U1.F1 (VDDSMPS): now also C28.1
- net +3V3A: now reaches U1.L1 (VDDA)
- net +3V3A: now also U1.M1 (VREF+), C64.1, C65.1
- net at U1.N17 (VCAPDSI): now also C34.1
- net SAI_SCK: now reaches U1.D1 (PE5)
- net SAI_FS: now reaches U1.D2 (PE4)
- net FMC_D7: now reaches U1.N9 (PE10)
- net FMC_D8: now reaches U1.P10 (PE11)
- net FMC_RS: now reaches U1.P7 (PF13)
- net I2C4_SCL: now reaches U1.P8 (PF14)
- net I2C4_SCL: now also R4.2
- net FMC_D6: now reaches U1.P9 (PE9)
- net FMC_D9: now reaches U1.R10 (PE12)
- net I2C4_SDA: now reaches U1.R9 (PF15)
- net I2C4_SDA: now also R3.2
- net FMC_D10: now reaches U1.T10 (PE13)
- net FMC_D5: now reaches U1.T9 (PE8)
- net FMC_D4: now reaches U1.U9 (PE7)
- net FMC_NWE: now reaches U1.A11 (PD5)
- net CAM_TIM: now reaches U1.A5 (PB5)
- net SAI_SD: now reaches U1.B11 (PD6)
- net CAM_RST: now reaches U1.B5 (PB6)
- net FMC_NE1: now reaches U1.C11 (PD7)
- net FMC_D2: now reaches U1.D13 (PD0)
- net FMC_D3: now reaches U1.E12 (PD1)
- net FMC_D1: now reaches U1.P15 (PD15)
- net FMC_D0: now reaches U1.P16 (PD14)
- net LCD_RST: now reaches U1.T15 (PB15)
- net FMC_D15: now reaches U1.T16 (PD10)
- net FMC_D14: now reaches U1.T17 (PD9)
- net TEAR: now reaches U1.U15 (PB14)
- net FMC_D13: now reaches U1.U16 (PD8)
- net LTDC_B3: no longer names the net of U1.B9 (PG11)
- net LTDC_B4: no longer names the net of U1.C8 (PK3)
- net LTDC_B5: no longer names the net of U1.A3 (PI5)
- net LTDC_B6: no longer names the net of U1.A8 (PK5)
- net LTDC_B7: no longer names the net of U1.C7 (PK6)
- net LTDC_CLK: no longer names the net of U1.F16 (PG7)
- net LTDC_DE: no longer names the net of U1.D7 (PK7)
- net LTDC_G2: no longer names the net of U1.D16 (PH13)
- net LTDC_G3: no longer names the net of U1.A9 (PG10)
- net LTDC_G4: no longer names the net of U1.B16 (PH15)
- net LTDC_G5: no longer names the net of U1.A16 (PI0)
- net LTDC_G7: no longer names the net of U1.B12 (PD3)
- net LTDC_HSYNC: no longer names the net of U1.F3 (PI10)
- net LTDC_R3: no longer names the net of U1.R13 (PH9)
- net LTDC_R4 renamed LIGHT_PWM
- net LTDC_R5: no longer names the net of U1.L2 (PC0)
- net LTDC_R6: no longer names the net of U1.E15 (PA8)
- net LTDC_R7: no longer names the net of U1.G14 (PG5)
- net LTDC_VSYNC: no longer names the net of U1.E2 (PI9)
- new net FMC_NOE: U1.A12 (PD4)
Other:
- note added: "FMC LCD"
- note added: "I2C"
- note added: "Power"
- note added: "SAI"
- note added: "USB"
- note added: "so basically everything should be 50 ohms"
- note removed: "LTDC"
- moved on the sheet: U1A, U1B, U1C, U1D, U1E

Commit message: almost finished power
Parts:
- renumbered C29 to C1, C53 to C10, C64 to C11, C36 to C12, C45 to C13, C54 to C14, C65 to C15, C37 to C16, C46 to C17, C55 to C18, C38 to C19, C34 to C2, C47 to C20, C56 to C21, C39 to C22, C48 to C23, C57 to C24, C40 to C25, C49 to C26, C58 to C27, C41 to C28, C50 to C29, C32 to C3, C59 to C30, C42 to C31, C51 to C32, C60 to C33, C43 to C34, C52 to C35, C61 to C36, C62 to C37, C63 to C38, C1 to C39, C28 to C4, C33 to C5, C30 to C6, C31 to C7, C35 to C8, C44 to C9, R2 to R1, R3 to R2, R4 to R3, R1 to R4, S2 to S1, S1 to S2

Commit message: PCB routed
Parts:
- added C89: 100n, Capacitor_SMD:C_0201_0603Metric, symbol Device:C
- added J7: Conn_ARM_JTAG_SWD_10, Connector_PinHeader_1.27mm:PinHeader_2x05_P1.27mm_Vertical_SMD, symbol Connector:Conn_ARM_JTAG_SWD_10
- C2: footprint Capacitor_SMD:C_0402_1005Metric -> Capacitor_SMD:C_0603_1608Metric
- L1: value 2.2u -> GNR4018S2R2MT; footprint (none) -> Inductor_SMD:L_Abracon_ASPI-4030S
Connections:
- net +3V3: now also U1.E7 (PDR_ON), C89.1, J7.1 (VTref)
- net DCMI_VSYNC: now also U1.A3 (PI5); no longer U1.A10 (PG9)
- net GND: now also C89.2, J7.3 (GND), J7.5 (GND), J7.9 (GNDDetect)
- net NRST: now also J7.10 (~{RESET})
- net SHDNZ: now reaches U1.B10 (PJ15)
- net RIGHT: now reaches U1.U6 (PJ3)
- net UP: now reaches U1.U7 (PJ4)
- net FMC_D12: now reaches U1.R11 (PE15)
- net FMC_D11: now reaches U1.U10 (PE14)
- net SWO: now reaches U1.R6 (PB2)
- net SWO: now also J7.6 (SWO/TDO)
- net TRIGGER: now reaches U1.U2 (PA3)
- net LEFT: now reaches U1.U3 (PA4)
- net DOWN: now reaches U1.U4 (PC5)
- net BUTTON: now reaches U1.U5 (PB0)
- net SWCLK: now reaches U1.B14 (SWCLK)
- net SWCLK: now also J7.4 (SWCLK/TCK)
- net SWDIO: now reaches U1.C15 (SWDIO)
- net SWDIO: now also J7.2 (SWDIO/TMS)
- no-connect marks 9 -> 118
Other:
- note added: "UI"

Commit message: finished r1 of the board
Parts:
- added R67: 22R, Resistor_SMD:R_0402_1005Metric, symbol Device:R
- C3, C5: footprint Capacitor_SMD:C_0402_1005Metric -> Capacitor_SMD:C_0603_1608Metric
Connections:
- net CAM_TIM: now also R67.1; no longer U1.A5 (PB5)
- new net: R67.2, U1.A5 (PB5)
Changed lines of the file:
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@@
 	(wire
 		(pts
+			(xy 31.75 83.82) (xy 36.83 83.82)
+		)
+		(stroke
+			(width 0)
+			(type default)
+		)
+	)
+	(wire
+		(pts
 			(xy 321.31 195.58) (xy 321.31 198.12)
 		)
@@
 	(wire
 		(pts
-			(xy 22.86 83.82) (xy 36.83 83.82)
+			(xy 13.97 83.82) (xy 24.13 83.82)
 		)
 		(stroke
@@
 	(wire
 		(pts
-			(xy 22.86 86.36) (xy 36.83 86.36)
+			(xy 13.97 86.36) (xy 36.83 86.36)
 		)
 		(stroke
@@
 	)
 	(label "CAM_RST"
-		(at 22.86 86.36 0)
+		(at 13.97 86.36 0)
 		(effects
 			(font
@@
 	)
 	(label "CAM_TIM"
-		(at 22.86 83.82 0)
+		(at 13.97 83.82 0)
 		(effects
 			(font
@@
 	)
 	(symbol
+		(lib_id "Device:R")
+		(at 27.94 83.82 90)
+		(unit 1)
+		(body_style 1)
+		(exclude_from_sim no)
+		(in_bom yes)
+		(on_board yes)
+		(in_pos_files yes)
+		(dnp no)
+		(property "Reference" "R67"
+			(at 27.94 78.994 90)
+			(show_name no)
+			(do_not_autoplace no)
+			(effects
+				(font
+					(size 1.27 1.27)
+				)
+			)
+		)
+		(property "Value" "22R"
+			(at 27.94 81.534 90)
+			(show_name no)
+			(do_not_autoplace no)
+			(effects
+				(font
+					(size 1.27 1.27)
+				)
+			)
+		)
+		(property "Footprint" "Resistor_SMD:R_0402_1005Metric"
+			(at 27.94 85.598 90)
+			(hide yes)
+			(show_name no)
+			(do_not_autoplace no)
+			(effects
+				(font
+					(size 1.27 1.27)
+				)
+			)
+		)
+		(property "Datasheet" ""
+			(at 27.94 83.82 0)
+			(hide yes)
+			(show_name no)
+			(do_not_autoplace no)
+			(effects
+				(font
+					(size 1.27 1.27)
+				)
+			)
+		)
+		(property "Description" "Resistor"
+			(at 27.94 83.82 0)
+			(hide yes)
+			(show_name no)
+			(do_not_autoplace no)
+			(effects
+				(font
+					(size 1.27 1.27)
+				)
+			)
+		)
+		(pin "1"
+		)
+		(pin "2"
+		)
+		(instances
+			(project "Microphone board"
+				(path "/54b36551-a175-45db-a91c-236f7d72a35b/d2dc67f8-a5f5-4154-8706-bc3e907f75c0"
+					(reference "R67")
+					(unit 1)
+				)
+			)
+		)
+	)
+	(symbol
 		(lib_id "Device:C")
 		(at 101.6 200.66 0)
@@
 			)
 		)
-		(property "Footprint" "Capacitor_SMD:C_0402_1005Metric"
+		(property "Footprint" "Capacitor_SMD:C_0603_1608Metric"
 			(at 102.5652 204.47 0)
 			(hide yes)
@@
 			)
 		)
-		(property "Footprint" "Capacitor_SMD:C_0402_1005Metric"
+		(property "Footprint" "Capacitor_SMD:C_0603_1608Metric"
 			(at 113.9952 204.47 0)
 			(hide yes)

Commit message: Updated project firmware
Parts:
- added D6: Red, PCM_JLCPCB:D_0603, symbol PCM_JLCPCB-Diodes:LED,0603,Red
- added R70: 470R, Resistor_SMD:R_0402_1005Metric, symbol Device:R
Connections:
- net GND: now also D6.1
- net STATUS_LED: now reaches U1.T3 (PA5)
- net STATUS_LED: now also R70.1
- new net: D6.2, R70.2
- no-connect marks 118 -> 117
Other:
- note added: "STATUS"
