File: Microphone board/MCU.kicad_sch (KiCad schematic)
At the start: 53 parts, among them J7 Conn_ARM_JTAG_SWD_10, U1 STM32H747XIH6, Y1 SX2M25.000M20F30TNN

Commit message: Syncing stuff between computers
Changed lines of the file:
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@@
+	(wire
+		(pts
+			(xy 119.38 39.37) (xy 133.35 39.37)
+		)
+		(stroke
+			(width 0)
+			(type default)
+		)
+	)
 	(wire
 		(pts
@@
 	(wire
 		(pts
+			(xy 119.38 41.91) (xy 133.35 41.91)
+		)
+		(stroke
+			(width 0)
+			(type default)
+		)
+	)
+	(wire
+		(pts
 			(xy 69.85 71.12) (xy 83.82 71.12)
 		)
@@
 	(wire
 		(pts
-			(xy 133.35 41.91) (xy 119.38 41.91)
-		)
-		(stroke
-			(width 0)
-			(type default)
-		)
-	)
-	(wire
-		(pts
 			(xy 82.55 248.92) (xy 82.55 246.38)
 		)
@@
 		)
 		(stroke
-			(width 0)
-			(type default)
-		)
-	)
-	(wire
-		(pts
-			(xy 133.35 39.37) (xy 119.38 39.37)
-		)
-		(stroke
