File: Microphone board/Microphone board.kicad_pcb (KiCad board)
At the start: 4 copper layers, 124.6 x 101 mm, 212 parts, among them J1 NHD-2.4-240320AF-CSXP, J2 OV2640, J3 TF-01A, J4 TYPE-C 16PIN 2MD(073), J5 Trigger, J6 Menu, J7 Conn_ARM_JTAG_SWD_10, M1 MSM261DDB019, M10 MSM261DDB019, M11 MSM261DDB019, M12 MSM261DDB019, M13 MSM261DDB019, M14 MSM261DDB019, M15 MSM261DDB019, M16 MSM261DDB019, M2 MSM261DDB019, M3 MSM261DDB019, M4 MSM261DDB019, M5 MSM261DDB019, M6 MSM261DDB019, M7 MSM261DDB019, M8 MSM261DDB019, M9 MSM261DDB019, Q1 MMBT3904, Q2 AO3401A, U1 STM32H747XIH6, U10 TPS7A2033PDBV, U11 USBLC6-2SC6, U2 24LC256, U3 TLV320ADC5140IRTWT, U4 TLV320ADC5140IRTWT, U5 TPD6F003, U6 TPS63001, U7 TPS2116DRL, U8 AP63203WU, U9 MCP73833-xxx-MF, Y1 SX2M25.000M20F30TNN

Commit message: Updated project firmware
Parts:
- added D6: Red, PCM_JLCPCB:D_0603, F.Cu at (144.8, 102.0)
- added R70: 470R, Resistor_SMD:R_0402_1005Metric, F.Cu at (144.8, 99.6)
- R39: footprint Resistor_SMD:R_0402_1005Metric -> Resistor_SMD:R_0603_1608Metric
- moved R39 0.30 mm to (165.0, 134.9)
- moved Q1 0.23 mm to (171.1, 137.5)
- moved Q2 0.23 mm to (165.1, 137.5)
- moved R35 0.23 mm to (174.6, 137.7)
- moved R36 0.23 mm to (173.6, 137.7)
- moved R37 0.23 mm to (168.1, 137.5)
- moved R38 0.23 mm to (168.1, 138.5)
Connections:
- J2 pad 8: unconnected-(J2-Pin_8-Pad8) -> GND
- U1 pad T3: unconnected-(U1C-PA5-PadT3) -> /MCU/STATUS_LED
Routing:
- net GND: track 36.4 -> 43.2 mm, vias 1528 -> 1537
- net /MCU/STATUS_LED: track 0.00 -> 4.38 mm
- net /Microphones/CH8_DAT: track 52.1 -> 51.0 mm
- net Net-(D6-Pad2): track 0.00 -> 1.11 mm
- net +3V3: vias 73 -> 68
Other:
- board text added: "STAT"
