File: Microphone board/Microphone board.kicad_pcb (KiCad board)
At the start: 4 copper layers, 124.6 x 101 mm, 214 parts, among them J1 NHD-2.4-240320AF-CSXP, J2 OV2640, J3 TF-01A, J4 TYPE-C 16PIN 2MD(073), J5 Trigger, J6 Menu, J7 Conn_ARM_JTAG_SWD_10, M1 MSM261DDB019, M10 MSM261DDB019, M11 MSM261DDB019, M12 MSM261DDB019, M13 MSM261DDB019, M14 MSM261DDB019, M15 MSM261DDB019, M16 MSM261DDB019, M2 MSM261DDB019, M3 MSM261DDB019, M4 MSM261DDB019, M5 MSM261DDB019, M6 MSM261DDB019, M7 MSM261DDB019, M8 MSM261DDB019, M9 MSM261DDB019, Q1 MMBT3904, Q2 AO3401A, U1 STM32H747XIH6, U10 TPS7A2033PDBV, U11 USBLC6-2SC6, U2 24LC256, U3 TLV320ADC5140IRTWT, U4 TLV320ADC5140IRTWT, U5 TPD6F003, U6 TPS63001, U7 TPS2116DRL, U8 AP63203WU, U9 MCP73833-xxx-MF, Y1 SX2M25.000M20F30TNN

Commit message: Syncing stuff between computers
Parts:
- removed R31, R32: 22R, Resistor_SMD:R_0402_1005Metric
Connections:
- U3 pad 22: Net-(U3A-BCLK) -> /MCU/SAI_SCK
- U3 pad 23: Net-(U3A-FSYNC) -> /MCU/SAI_FS
Routing:
- net /MCU/SAI_SCK: track 21.0 -> 23.1 mm, vias 2 -> 3
- net /MCU/SAI_FS: track 22.7 -> 24.5 mm, vias 2 -> 3
- net Net-(U3A-FSYNC): track 1.39 -> 0.00 mm
- net Net-(U3A-BCLK): track 1.36 -> 0.00 mm
- net /MCU/DCMI_D6: track 51.3 -> 52.2 mm
- net GND: vias 1537 -> 1540
