File: Microphone board/camera.kicad_sch (KiCad schematic)
At the start: 0 parts

Commit message: Made almost the rest of the schematic lol
Parts:
- added C66, C67, C70: 100n, Capacitor_SMD:C_0402_1005Metric, symbol Device:C
- added C68, C71: 4.7u, Capacitor_SMD:C_0603_1608Metric, symbol Device:C
- added J2: OV2640, Connector_FFC-FPC:Amphenol_F32R-1A7x1-11024_1x24-1MP_P0.5mm_Horizontal, symbol Connector_Generic_MountingPin:Conn_01x24_MountingPin
- added R42: 10k, Resistor_SMD:R_0402_1005Metric, symbol Device:R
Connections:
- new net: J2.1 (Pin_1), R42.2
- new net +3V3: C66.1, C67.1, C68.1, J2.10 (Pin_10), J2.11 (Pin_11)
- new net +3V3A: C70.1, C71.1, J2.4 (Pin_4)
- new net DCMI_D0: J2.19 (Pin_19)
- new net DCMI_D1: J2.21 (Pin_21)
- new net DCMI_D2: J2.22 (Pin_22)
- new net DCMI_D3: J2.20 (Pin_20)
- new net DCMI_D5: J2.16 (Pin_16)
- new net DCMI_D6: J2.14 (Pin_14)
- new net DCMI_D7: J2.12 (Pin_12), J2.18 (Pin_18)
- new net DCMI_HSYNC: J2.9 (Pin_9)
- new net DCMI_PIXCLK: J2.17 (Pin_17)
- new net DCMI_VSYNC: J2.7 (Pin_7)
- new net GND: C66.2, C67.2, C68.2, C70.2, C71.2, J2.15 (Pin_15), J2.2 (Pin_2), J2.MP (MountPin), R42.1
- new net RST: J2.6 (Pin_6)
- new net SCL: J2.5 (Pin_5)
- new net SDA: J2.3 (Pin_3)
- new net TIM: J2.13 (Pin_13)
- no-connect marks 0 -> 3

Commit message: almost finished power
Parts:
- renumbered C66 to C72, C67 to C73, C68 to C74, R42 to R40
Changed lines of the file:
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@@
 		(dnp no)
 		(fields_autoplaced yes)
-		(property "Reference" "R42"
+		(property "Reference" "R40"
 			(at 195.58 54.61 90)
 			(show_name no)
@@
 			(project "Microphone board"
 				(path "/54b36551-a175-45db-a91c-236f7d72a35b/610e6e28-9b6e-4cdb-9ff1-31672a321cfc"
-					(reference "R42")
+					(reference "R40")
 					(unit 1)
 				)
@@
 		(dnp no)
 		(fields_autoplaced yes)
-		(property "Reference" "#PWR098"
+		(property "Reference" "#PWR097"
 			(at 100.33 73.66 0)
 			(hide yes)
@@
 			(project "Microphone board"
 				(path "/54b36551-a175-45db-a91c-236f7d72a35b/610e6e28-9b6e-4cdb-9ff1-31672a321cfc"
-					(reference "#PWR098")
+					(reference "#PWR097")
 					(unit 1)
 				)
@@
 		(dnp no)
 		(fields_autoplaced yes)
-		(property "Reference" "C66"
+		(property "Reference" "C72"
 			(at 129.54 77.4699 0)
 			(show_name no)
@@
 			(project "Microphone board"
 				(path "/54b36551-a175-45db-a91c-236f7d72a35b/610e6e28-9b6e-4cdb-9ff1-31672a321cfc"
-					(reference "C66")
+					(reference "C72")
 					(unit 1)
 				)
@@
 		(dnp no)
 		(fields_autoplaced yes)
-		(property "Reference" "#PWR092"
+		(property "Reference" "#PWR0104"
 			(at 218.44 133.35 0)
 			(hide yes)
@@
 			(project "Microphone board"
 				(path "/54b36551-a175-45db-a91c-236f7d72a35b/610e6e28-9b6e-4cdb-9ff1-31672a321cfc"
-					(reference "#PWR092")
+					(reference "#PWR0104")
 					(unit 1)
 				)
@@
 		(dnp no)
 		(fields_autoplaced yes)
-		(property "Reference" "#PWR097"
+		(property "Reference" "#PWR0100"
 			(at 148.59 93.98 0)
 			(hide yes)
@@
 			(project "Microphone board"
 				(path "/54b36551-a175-45db-a91c-236f7d72a35b/610e6e28-9b6e-4cdb-9ff1-31672a321cfc"
-					(reference "#PWR097")
+					(reference "#PWR0100")
 					(unit 1)
 				)
@@
 		(dnp no)
 		(fields_autoplaced yes)
-		(property "Reference" "#PWR099"
+		(property "Reference" "#PWR098"
 			(at 111.76 93.98 0)
 			(hide yes)
@@
 			(project "Microphone board"
 				(path "/54b36551-a175-45db-a91c-236f7d72a35b/610e6e28-9b6e-4cdb-9ff1-31672a321cfc"
-					(reference "#PWR099")
+					(reference "#PWR098")
 					(unit 1)
 				)
@@
 		(dnp no)
 		(fields_autoplaced yes)
-		(property "Reference" "C67"
+		(property "Reference" "C73"
 			(at 140.97 77.4699 0)
 			(show_name no)
@@
 			(project "Microphone board"
 				(path "/54b36551-a175-45db-a91c-236f7d72a35b/610e6e28-9b6e-4cdb-9ff1-31672a321cfc"
-					(reference "C67")
+					(reference "C73")
 					(unit 1)
 				)
@@
 		(dnp no)
 		(fields_autoplaced yes)
-		(property "Reference" "#PWR094"
+		(property "Reference" "#PWR0102"
 			(at 208.28 62.23 0)
 			(hide yes)
@@
 			(project "Microphone board"
 				(path "/54b36551-a175-45db-a91c-236f7d72a35b/610e6e28-9b6e-4cdb-9ff1-31672a321cfc"
-					(reference "#PWR094")
+					(reference "#PWR0102")
 					(unit 1)
 				)
@@
 		(dnp no)
 		(fields_autoplaced yes)
-		(property "Reference" "#PWR096"
+		(property "Reference" "#PWR099"
 			(at 125.73 73.66 0)
 			(hide yes)
@@
 			(project "Microphone board"
 				(path "/54b36551-a175-45db-a91c-236f7d72a35b/610e6e28-9b6e-4cdb-9ff1-31672a321cfc"
-					(reference "#PWR096")
+					(reference "#PWR099")
 					(unit 1)
 				)
@@
 		(dnp no)
 		(fields_autoplaced yes)
-		(property "Reference" "#PWR093"
+		(property "Reference" "#PWR0103"
 			(at 210.82 133.35 0)
 			(hide yes)
@@
 			(project "Microphone board"
 				(path "/54b36551-a175-45db-a91c-236f7d72a35b/610e6e28-9b6e-4cdb-9ff1-31672a321cfc"
-					(reference "#PWR093")
+					(reference "#PWR0103")
 					(unit 1)
 				)
@@
 		(dnp no)
 		(fields_autoplaced yes)
-		(property "Reference" "#PWR095"
+		(property "Reference" "#PWR0101"
 			(at 201.93 62.23 0)
 			(hide yes)
@@
 			(project "Microphone board"
 				(path "/54b36551-a175-45db-a91c-236f7d72a35b/610e6e28-9b6e-4cdb-9ff1-31672a321cfc"
-					(reference "#PWR095")
+					(reference "#PWR0101")
 					(unit 1)
 				)
@@
 		(dnp no)
 		(fields_autoplaced yes)
-		(property "Reference" "C68"
+		(property "Reference" "C74"
 			(at 152.4 77.4699 0)
 			(show_name no)
@@
 			(project "Microphone board"
 				(path "/54b36551-a175-45db-a91c-236f7d72a35b/610e6e28-9b6e-4cdb-9ff1-31672a321cfc"
-					(reference "C68")
-					(unit 1)
-				)
+					(reference "C74")
+					(unit 1)
+				)

Commit message: PCB routed
Parts:
- added C90: OV2640, Mic_Parts:OV2640, symbol Mic_Parts:OV2640_base
- J2: footprint Connector_FFC-FPC:Amphenol_F32R-1A7x1-11024_1x24-1MP_P0.5mm_Horizontal -> Connector_FFC-FPC:Amphenol_F32Q-1A7x1-11024_1x24-1MP_P0.5mm_Horizontal
Connections:
- net DCMI_D7: no longer J2.18 (Pin_18)
- new net DCMI_D4: J2.18 (Pin_18)
Changed lines of the file:
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@@
 		)
 	)
-	(label "DCMI_D7"
+	(label "DCMI_D4"
 		(at 175.26 104.14 0)
 		(effects
@@
 	)
 	(symbol
+		(lib_id "Mic_Parts:OV2640_base")
+		(at 234.95 69.85 0)
+		(unit 1)
+		(body_style 1)
+		(exclude_from_sim no)
+		(in_bom yes)
+		(on_board yes)
+		(in_pos_files yes)
+		(dnp no)
+		(fields_autoplaced yes)
+		(property "Reference" "C90"
+			(at 238.76 68.5799 0)
+			(show_name no)
+			(do_not_autoplace no)
+			(effects
+				(font
+					(size 1.27 1.27)
+				)
+				(justify left)
+			)
+		)
+		(property "Value" "OV2640"
+			(at 238.76 71.1199 0)
+			(show_name no)
+			(do_not_autoplace no)
+			(effects
+				(font
+					(size 1.27 1.27)
+				)
+				(justify left)
+			)
+		)
+		(property "Footprint" "Mic_Parts:OV2640"
+			(at 234.95 69.85 0)
+			(hide yes)
+			(show_name no)
+			(do_not_autoplace no)
+			(effects
+				(font
+					(size 1.27 1.27)
+				)
+			)
+		)
+		(property "Datasheet" "https://www.arducam.com/arducam-ov2640-camera-module-2mp-mini-ccm-compact-camera-modules-compatible-with-arduino_m0031esp32-esp8266-development-board-with-dvp-24-pin-interface_.html"
+			(at 235.204 69.596 0)
+			(hide yes)
+			(show_name no)
+			(do_not_autoplace no)
+			(effects
+				(font
+					(size 1.27 1.27)
+				)
+			)
+		)
+		(property "Description" ""
+			(at 234.95 69.85 0)
+			(hide yes)
+			(show_name no)
+			(do_not_autoplace no)
+			(effects
+				(font
+					(size 1.27 1.27)
+				)
+			)
+		)
+		(instances
+			(project "Microphone board"
+				(path "/54b36551-a175-45db-a91c-236f7d72a35b/610e6e28-9b6e-4cdb-9ff1-31672a321cfc"
+					(reference "C90")
+					(unit 1)
+				)
+			)
+		)
+	)
+	(symbol
 		(lib_id "Device:C")
 		(at 125.73 78.74 0)
@@
 			)
 		)
-		(property "Footprint" "Connector_FFC-FPC:Amphenol_F32R-1A7x1-11024_1x24-1MP_P0.5mm_Horizontal"
+		(property "Footprint" "Connector_FFC-FPC:Amphenol_F32Q-1A7x1-11024_1x24-1MP_P0.5mm_Horizontal"
 			(at 218.44 88.9 0)
 			(hide yes)

Commit message: finished r1 of the board
Parts:
- J2: footprint Connector_FFC-FPC:Amphenol_F32Q-1A7x1-11024_1x24-1MP_P0.5mm_Horizontal -> Connector_FFC-FPC:Hirose_FH12-24S-0.5SH_1x24-1MP_P0.50mm_Horizontal
Changed lines of the file:
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@@
 			)
 		)
-		(property "Footprint" "Connector_FFC-FPC:Amphenol_F32Q-1A7x1-11024_1x24-1MP_P0.5mm_Horizontal"
+		(property "Footprint" "Connector_FFC-FPC:Hirose_FH12-24S-0.5SH_1x24-1MP_P0.50mm_Horizontal"
 			(at 218.44 88.9 0)
 			(hide yes)

Commit message: Updated project firmware
Connections:
- net GND: now also J2.8 (Pin_8)
- no-connect marks 3 -> 2
Changed lines of the file:
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@@
+	)
+	(junction
+		(at 210.82 78.74)
+		(diameter 0)
+		(color 0 0 0 0)
 	)
 	(junction
@@
 	)
 	(no_connect
-		(at 213.36 78.74)
-	)
-	(no_connect
 		(at 213.36 116.84)
 	)
@@
 	(wire
 		(pts
+			(xy 210.82 78.74) (xy 210.82 96.52)
+		)
+		(stroke
+			(width 0)
+			(type default)
+		)
+	)
+	(wire
+		(pts
 			(xy 210.82 96.52) (xy 210.82 127)
 		)
@@
 	(wire
 		(pts
-			(xy 210.82 63.5) (xy 210.82 96.52)
+			(xy 210.82 63.5) (xy 210.82 78.74)
 		)
 		(stroke
@@
 		)
 		(stroke
+			(width 0)
+			(type default)
+		)
+	)
+	(wire
+		(pts
+			(xy 210.82 78.74) (xy 213.36 78.74)
+		)
+		(stroke
