File: Microphone board/display.kicad_sch (KiCad schematic)
At the start: 0 parts

Commit message: Made almost the rest of the schematic lol
Parts:
- added C72, C73: 100n, Capacitor_SMD:C_0402_1005Metric, symbol Device:C
- added C74: 4.7u, Capacitor_SMD:C_0603_1608Metric, symbol Device:C
- added J3: NHD-2.4-240320AF-CSXP, Connector_FFC-FPC:Amphenol_F32R-1A7x1-11040_1x40-1MP_P0.5mm_Horizontal, symbol Connector_Generic_MountingPin:Conn_01x40_MountingPin
- added Q1: AO3401A, PCM_Package_TO_SOT_SMD_AKL:SOT-23, symbol PCM_Transistor_MOSFET_AKL:AO3401A
- added Q2: MMBT3904, PCM_Package_TO_SOT_SMD_AKL:SOT-23, symbol PCM_Transistor_BJT_AKL:MMBT3904
- added R44: 10R, Resistor_SMD:R_0402_1005Metric, symbol Device:R
- added R45: 4k7, Resistor_SMD:R_0402_1005Metric, symbol Device:R
- added R46: 2R, Resistor_SMD:R_0402_1005Metric, symbol Device:R
- added R47: 1k, Resistor_SMD:R_0402_1005Metric, symbol Device:R
- added R48: 10k, Resistor_SMD:R_0402_1005Metric, symbol Device:R
Connections:
- new net: Q2.3 (C), R44.1, R45.1
- new net: Q1.1 (G), R44.2
- new net: Q2.1 (B), R47.2, R48.2
- new net: Q1.3 (D), R46.1
- new net +3V3: C72.1, C73.1, C74.1, J3.7 (Pin_7), J3.8 (Pin_8), Q1.2 (S), R45.2
- new net FMC_D0: J3.14 (Pin_14)
- new net FMC_D1: J3.15 (Pin_15)
- new net FMC_D10: J3.24 (Pin_24)
- new net FMC_D11: J3.25 (Pin_25)
- new net FMC_D12: J3.26 (Pin_26)
- new net FMC_D13: J3.27 (Pin_27)
- new net FMC_D14: J3.28 (Pin_28)
- new net FMC_D15: J3.29 (Pin_29)
- new net FMC_D2: J3.16 (Pin_16)
- new net FMC_D3: J3.17 (Pin_17)
- new net FMC_D4: J3.18 (Pin_18)
- new net FMC_D5: J3.19 (Pin_19)
- new net FMC_D6: J3.20 (Pin_20)
- new net FMC_D7: J3.21 (Pin_21)
- new net FMC_D8: J3.22 (Pin_22)
- new net FMC_D9: J3.23 (Pin_23)
- new net FMC_NOE: J3.13 (Pin_13)
- new net FMC_NWE: J3.12 (Pin_12)
- new net FMC_RS: J3.11 (Pin_11)
- new net GND: C72.2, C73.2, C74.2, J3.1 (Pin_1), J3.10 (Pin_10), J3.31 (Pin_31), J3.32 (Pin_32), J3.33 (Pin_33), J3.34 (Pin_34), J3.35 (Pin_35), J3.36 (Pin_36), J3.37 (Pin_37), J3.39 (Pin_39), J3.9 (Pin_9), J3.MP (MountPin), Q2.2 (E), R48.1
- new net LIGHT: J3.38 (Pin_38), R46.2
- new net LIGHT_PWM: R47.1
- new net RST: J3.30 (Pin_30)
- new net TEAR: J3.40 (Pin_40)
- no-connect marks 0 -> 5

Commit message: almost finished power
Parts:
- renumbered C72 to C67, C73 to C68, C74 to C69, J3 to J1, Q2 to Q1, Q1 to Q2, R47 to R35, R48 to R36, R45 to R37, R44 to R38, R46 to R39
Changed lines of the file:
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@@
 		(dnp no)
 		(fields_autoplaced yes)
-		(property "Reference" "C74"
+		(property "Reference" "C69"
 			(at 157.48 80.0099 0)
 			(show_name no)
@@
 			(project "Microphone board"
 				(path "/54b36551-a175-45db-a91c-236f7d72a35b/933df564-ce74-4453-93df-6ff071652f89"
-					(reference "C74")
+					(reference "C69")
 					(unit 1)
 				)
@@
 		(dnp no)
 		(fields_autoplaced yes)
-		(property "Reference" "#PWR0109"
+		(property "Reference" "#PWR092"
 			(at 128.27 76.2 0)
 			(hide yes)
@@
 			(project "Microphone board"
 				(path "/54b36551-a175-45db-a91c-236f7d72a35b/933df564-ce74-4453-93df-6ff071652f89"
-					(reference "#PWR0109")
+					(reference "#PWR092")
 					(unit 1)
 				)
@@
 		(dnp no)
 		(fields_autoplaced yes)
-		(property "Reference" "R44"
+		(property "Reference" "R38"
 			(at 67.31 81.28 90)
 			(show_name no)
@@
 			(project "Microphone board"
 				(path "/54b36551-a175-45db-a91c-236f7d72a35b/933df564-ce74-4453-93df-6ff071652f89"
-					(reference "R44")
+					(reference "R38")
 					(unit 1)
 				)
@@
 		(dnp no)
 		(fields_autoplaced yes)
-		(property "Reference" "R48"
+		(property "Reference" "R36"
 			(at 53.34 100.3299 0)
 			(show_name no)
@@
 			(project "Microphone board"
 				(path "/54b36551-a175-45db-a91c-236f7d72a35b/933df564-ce74-4453-93df-6ff071652f89"
-					(reference "R48")
+					(reference "R36")
 					(unit 1)
 				)
@@
 		(dnp no)
 		(fields_autoplaced yes)
-		(property "Reference" "R46"
+		(property "Reference" "R39"
 			(at 82.55 99.0599 0)
 			(show_name no)
@@
 			(project "Microphone board"
 				(path "/54b36551-a175-45db-a91c-236f7d72a35b/933df564-ce74-4453-93df-6ff071652f89"
-					(reference "R46")
+					(reference "R39")
 					(unit 1)
 				)
@@
 		(dnp no)
 		(fields_autoplaced yes)
-		(property "Reference" "#PWR0103"
+		(property "Reference" "#PWR090"
 			(at 60.96 76.2 0)
 			(hide yes)
@@
 			(project "Microphone board"
 				(path "/54b36551-a175-45db-a91c-236f7d72a35b/933df564-ce74-4453-93df-6ff071652f89"
-					(reference "#PWR0103")
+					(reference "#PWR090")
 					(unit 1)
 				)
@@
 		(dnp no)
 		(fields_autoplaced yes)
-		(property "Reference" "Q1"
+		(property "Reference" "Q2"
 			(at 83.82 87.6299 0)
 			(show_name no)
@@
 			(project "Microphone board"
 				(path "/54b36551-a175-45db-a91c-236f7d72a35b/933df564-ce74-4453-93df-6ff071652f89"
-					(reference "Q1")
+					(reference "Q2")
 					(unit 1)
 				)
@@
 		(dnp no)
 		(fields_autoplaced yes)
-		(property "Reference" "R47"
+		(property "Reference" "R35"
 			(at 44.45 88.9 90)
 			(show_name no)
@@
 			(project "Microphone board"
 				(path "/54b36551-a175-45db-a91c-236f7d72a35b/933df564-ce74-4453-93df-6ff071652f89"
-					(reference "R47")
+					(reference "R35")
 					(unit 1)
 				)
@@
 		(dnp no)
 		(fields_autoplaced yes)
-		(property "Reference" "#PWR0105"
+		(property "Reference" "#PWR091"
 			(at 60.96 114.3 0)
 			(hide yes)
@@
 			(project "Microphone board"
 				(path "/54b36551-a175-45db-a91c-236f7d72a35b/933df564-ce74-4453-93df-6ff071652f89"
-					(reference "#PWR0105")
+					(reference "#PWR091")
 					(unit 1)
 				)
@@
 		(dnp no)
 		(fields_autoplaced yes)
-		(property "Reference" "#PWR0104"
+		(property "Reference" "#PWR089"
 			(at 50.8 114.3 0)
 			(hide yes)
@@
 			(project "Microphone board"
 				(path "/54b36551-a175-45db-a91c-236f7d72a35b/933df564-ce74-4453-93df-6ff071652f89"
-					(reference "#PWR0104")
+					(reference "#PWR089")
 					(unit 1)
 				)
@@
 		(dnp no)
 		(fields_autoplaced yes)
-		(property "Reference" "#PWR0101"
+		(property "Reference" "#PWR095"
 			(at 191.77 148.59 0)
 			(hide yes)
@@
 			(project "Microphone board"
 				(path "/54b36551-a175-45db-a91c-236f7d72a35b/933df564-ce74-4453-93df-6ff071652f89"
-					(reference "#PWR0101")
+					(reference "#PWR095")
 					(unit 1)
 				)
@@
 		(dnp no)
 		(fields_autoplaced yes)
-		(property "Reference" "Q2"
+		(property "Reference" "Q1"
 			(at 63.5 93.9799 0)
 			(show_name no)
@@
 			(project "Microphone board"
 				(path "/54b36551-a175-45db-a91c-236f7d72a35b/933df564-ce74-4453-93df-6ff071652f89"
-					(reference "Q2")
+					(reference "Q1")
 					(unit 1)
 				)
@@
 		(in_pos_files yes)
 		(dnp no)
-		(property "Reference" "R45"
+		(property "Reference" "R37"
 			(at 58.42 80.0099 0)
 			(show_name no)
@@
 			(project "Microphone board"
 				(path "/54b36551-a175-45db-a91c-236f7d72a35b/933df564-ce74-4453-93df-6ff071652f89"
-					(reference "R45")
+					(reference "R37")
 					(unit 1)
 				)
@@
 		(dnp no)
 		(fields_autoplaced yes)
-		(property "Reference" "C72"
+		(property "Reference" "C67"
 			(at 132.08 80.0099 0)
 			(show_name no)
@@
 			(project "Microphone board"
 				(path "/54b36551-a175-45db-a91c-236f7d72a35b/933df564-ce74-4453-93df-6ff071652f89"
-					(reference "C72")
+					(reference "C67")
 					(unit 1)
 				)
@@
 		(dnp no)
 		(fields_autoplaced yes)
-		(property "Reference" "#PWR0102"
+		(property "Reference" "#PWR094"
 			(at 189.23 39.37 0)
 			(hide yes)
@@
 			(project "Microphone board"
 				(path "/54b36551-a175-45db-a91c-236f7d72a35b/933df564-ce74-4453-93df-6ff071652f89"
-					(reference "#PWR0102")
+					(reference "#PWR094")
 					(unit 1)
 				)
@@
 		(dnp no)
 		(fields_autoplaced yes)
-		(property "Reference" "J3"
+		(property "Reference" "J1"
 			(at 201.93 84.1755 0)
 			(show_name no)
@@
 			(project "Microphone board"
 				(path "/54b36551-a175-45db-a91c-236f7d72a35b/933df564-ce74-4453-93df-6ff071652f89"
-					(reference "J3")
+					(reference "J1")
 					(unit 1)
 				)
@@
 		(dnp no)
 		(fields_autoplaced yes)
-		(property "Reference" "C73"
+		(property "Reference" "C68"
 			(at 144.78 80.0099 0)
 			(show_name no)
@@
 			(project "Microphone board"
 				(path "/54b36551-a175-45db-a91c-236f7d72a35b/933df564-ce74-4453-93df-6ff071652f89"
-					(reference "C73")
+					(reference "C68")
 					(unit 1)
 				)
@@
 		(dnp no)
 		(fields_autoplaced yes)
-		(property "Reference" "#PWR0108"
+		(property "Reference" "#PWR093"
 			(at 153.67 96.52 0)
 			(hide yes)
@@
 			(project "Microphone board"
 				(path "/54b36551-a175-45db-a91c-236f7d72a35b/933df564-ce74-4453-93df-6ff071652f89"
-					(reference "#PWR0108")
+					(reference "#PWR093")
 					(unit 1)
 				)
@@
 		(dnp no)
 		(fields_autoplaced yes)
-		(property "Reference" "#PWR0100"
+		(property "Reference" "#PWR096"
 			(at 199.39 148.59 0)
 			(hide yes)
@@
 			(project "Microphone board"
 				(path "/54b36551-a175-45db-a91c-236f7d72a35b/933df564-ce74-4453-93df-6ff071652f89"
-					(reference "#PWR0100")
-					(unit 1)
-				)
+					(reference "#PWR096")
+					(unit 1)
+				)

Commit message: PCB routed
Connections:
- net +3V3: now also J1.33 (Pin_33), J1.34 (Pin_34); no longer J1.7 (Pin_7), J1.8 (Pin_8)
- net FMC_D0: now also J1.27 (Pin_27); no longer J1.14 (Pin_14)
- net FMC_D1: now also J1.26 (Pin_26); no longer J1.15 (Pin_15)
- net FMC_D10: now also J1.17 (Pin_17); no longer J1.24 (Pin_24)
- net FMC_D11: now also J1.16 (Pin_16); no longer J1.25 (Pin_25)
- net FMC_D12: now also J1.15 (Pin_15); no longer J1.26 (Pin_26)
- net FMC_D13: now also J1.14 (Pin_14); no longer J1.27 (Pin_27)
- net FMC_D14: now also J1.13 (Pin_13); no longer J1.28 (Pin_28)
- net FMC_D15: now also J1.12 (Pin_12); no longer J1.29 (Pin_29)
- net FMC_D2: now also J1.25 (Pin_25); no longer J1.16 (Pin_16)
- net FMC_D3: now also J1.24 (Pin_24); no longer J1.17 (Pin_17)
- net FMC_D4: now also J1.23 (Pin_23); no longer J1.18 (Pin_18)
- net FMC_D5: now also J1.22 (Pin_22); no longer J1.19 (Pin_19)
- net FMC_D6: now also J1.21 (Pin_21); no longer J1.20 (Pin_20)
- net FMC_D7: now also J1.20 (Pin_20); no longer J1.21 (Pin_21)
- net FMC_D8: now also J1.19 (Pin_19); no longer J1.22 (Pin_22)
- net FMC_D9: now also J1.18 (Pin_18); no longer J1.23 (Pin_23)
- net FMC_NOE: now also J1.28 (Pin_28); no longer J1.13 (Pin_13)
- net FMC_NWE: now also J1.29 (Pin_29); no longer J1.12 (Pin_12)
- net FMC_RS: now also J1.30 (Pin_30); no longer J1.11 (Pin_11)
- net GND: now also J1.2 (Pin_2), J1.4 (Pin_4), J1.40 (Pin_40), J1.5 (Pin_5), J1.6 (Pin_6), J1.7 (Pin_7), J1.8 (Pin_8); no longer J1.1 (Pin_1), J1.33 (Pin_33), J1.34 (Pin_34), J1.35 (Pin_35), J1.36 (Pin_36), J1.37 (Pin_37), J1.39 (Pin_39)
- net LIGHT: now also J1.3 (Pin_3); no longer J1.38 (Pin_38)
- net RST: now also J1.11 (Pin_11); no longer J1.30 (Pin_30)
- net TEAR: now also J1.1 (Pin_1); no longer J1.40 (Pin_40)
Changed lines of the file:
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@@
+	(wire
+		(pts
+			(xy 199.39 30.48) (xy 199.39 27.94)
+		)
+		(stroke
+			(width 0)
+			(type default)
+		)
+	)
 	(wire
 		(pts
@@
 	(wire
 		(pts
+			(xy 199.39 27.94) (xy 204.47 27.94)
+		)
+		(stroke
+			(width 0)
+			(type default)
+		)
+	)
+	(wire
+		(pts
 			(xy 191.77 124.46) (xy 191.77 127)
 		)
@@
 	(wire
 		(pts
-			(xy 199.39 139.7) (xy 199.39 142.24)
+			(xy 204.47 27.94) (xy 204.47 30.48)
 		)
 		(stroke
@@
 	)
 	(symbol
+		(lib_id "Connector_Generic_MountingPin:Conn_01x40_MountingPin")
+		(at 199.39 86.36 0)
+		(mirror x)
+		(unit 1)
+		(body_style 1)
+		(exclude_from_sim no)
+		(in_bom yes)
+		(on_board yes)
+		(in_pos_files yes)
+		(dnp no)
+		(property "Reference" "J1"
+			(at 201.93 86.0045 0)
+			(show_name no)
+			(do_not_autoplace no)
+			(effects
+				(font
+					(size 1.27 1.27)
+				)
+				(justify left)
+			)
+		)
+		(property "Value" "NHD-2.4-240320AF-CSXP"
+			(at 201.93 83.4645 0)
+			(show_name no)
+			(do_not_autoplace no)
+			(effects
+				(font
+					(size 1.27 1.27)
+				)
+				(justify left)
+			)
+		)
+		(property "Footprint" "Connector_FFC-FPC:Amphenol_F32R-1A7x1-11040_1x40-1MP_P0.5mm_Horizontal"
+			(at 199.39 86.36 0)
+			(hide yes)
+			(show_name no)
+			(do_not_autoplace no)
+			(effects
+				(font
+					(size 1.27 1.27)
+				)
+			)
+		)
+		(property "Datasheet" ""
+			(at 199.39 86.36 0)
+			(hide yes)
+			(show_name no)
+			(do_not_autoplace no)
+			(effects
+				(font
+					(size 1.27 1.27)
+				)
+			)
+		)
+		(property "Description" "Generic connectable mounting pin connector, single row, 01x40, script generated (kicad-library-utils/schlib/autogen/connector/)"
+			(at 199.39 86.36 0)
+			(hide yes)
+			(show_name no)
+			(do_not_autoplace no)
+			(effects
+				(font
+					(size 1.27 1.27)
+				)
+			)
+		)
+		(pin "8"
+		)
+		(pin "9"
+		)
+		(pin "2"
+		)
+		(pin "15"
+		)
+		(pin "20"
+		)
+		(pin "11"
+		)
+		(pin "28"
+		)
+		(pin "30"
+		)
+		(pin "31"
+		)
+		(pin "18"
+		)
+		(pin "1"
+		)
+		(pin "6"
+		)
+		(pin "21"
+		)
+		(pin "4"
+		)
+		(pin "22"
+		)
+		(pin "5"
+		)
+		(pin "23"
+		)
+		(pin "25"
+		)
+		(pin "14"
+		)
+		(pin "3"
+		)
+		(pin "16"
+		)
+		(pin "26"
+		)
+		(pin "7"
+		)
+		(pin "10"
+		)
+		(pin "12"
+		)
+		(pin "19"
+		)
+		(pin "13"
+		)
+		(pin "17"
+		)
+		(pin "24"
+		)
+		(pin "27"
+		)
+		(pin "29"
+		)
+		(pin "37"
+		)
+		(pin "40"
+		)
+		(pin "MP"
+		)
+		(pin "39"
+		)
+		(pin "33"
+		)
+		(pin "34"
+		)
+		(pin "35"
+		)
+		(pin "36"
+		)
+		(pin "32"
+		)
+		(pin "38"
+		)
+		(instances
+			(project "Microphone board"
+				(path "/54b36551-a175-45db-a91c-236f7d72a35b/933df564-ce74-4453-93df-6ff071652f89"
+					(reference "J1")
+					(unit 1)
+				)
+			)
+		)
+	)
+	(symbol
 		(lib_id "PCM_Transistor_MOSFET_AKL:AO3401A")
 		(at 77.47 88.9 0)
@@
 	)
 	(symbol
-		(lib_id "Connector_Generic_MountingPin:Conn_01x40_MountingPin")
-		(at 199.39 83.82 0)
-		(unit 1)
-		(body_style 1)
-		(exclude_from_sim no)
-		(in_bom yes)
-		(on_board yes)
-		(in_pos_files yes)
-		(dnp no)
-		(fields_autoplaced yes)
-		(property "Reference" "J1"
-			(at 201.93 84.1755 0)
-			(show_name no)
-			(do_not_autoplace no)
-			(effects
-				(font
-					(size 1.27 1.27)
-				)
-				(justify left)
-			)
-		)
-		(property "Value" "NHD-2.4-240320AF-CSXP"
-			(at 201.93 86.7155 0)
-			(show_name no)
-			(do_not_autoplace no)
-			(effects
-				(font
-					(size 1.27 1.27)
-				)
-				(justify left)
-			)
-		)
-		(property "Footprint" "Connector_FFC-FPC:Amphenol_F32R-1A7x1-11040_1x40-1MP_P0.5mm_Horizontal"
-			(at 199.39 83.82 0)
-			(hide yes)
-			(show_name no)
-			(do_not_autoplace no)
-			(effects
-				(font
-					(size 1.27 1.27)
-				)
-			)
-		)
-		(property "Datasheet" ""
-			(at 199.39 83.82 0)
-			(hide yes)
-			(show_name no)
-			(do_not_autoplace no)
-			(effects
-				(font
-					(size 1.27 1.27)
-				)
-			)
-		)
-		(property "Description" "Generic connectable mounting pin connector, single row, 01x40, script generated (kicad-library-utils/schlib/autogen/connector/)"
-			(at 199.39 83.82 0)
-			(hide yes)
-			(show_name no)
-			(do_not_autoplace no)
-			(effects
-				(font
-					(size 1.27 1.27)
-				)
-			)
-		)
-		(pin "8"
-		)
-		(pin "9"
-		)
-		(pin "2"
-		)
-		(pin "15"
-		)
-		(pin "20"
-		)
-		(pin "11"
-		)
-		(pin "28"
-		)
-		(pin "30"
-		)
-		(pin "31"
-		)
-		(pin "18"
-		)
-		(pin "1"
-		)
-		(pin "6"
-		)
-		(pin "21"
-		)
-		(pin "4"
-		)
-		(pin "22"
-		)
-		(pin "5"
-		)
-		(pin "23"
-		)
-		(pin "25"
-		)
-		(pin "14"
-		)
-		(pin "3"
-		)
-		(pin "16"
-		)
-		(pin "26"
-		)
-		(pin "7"
-		)
-		(pin "10"
-		)
-		(pin "12"
-		)
-		(pin "19"
-		)
-		(pin "13"
-		)
-		(pin "17"
-		)
-		(pin "24"
-		)
-		(pin "27"
-		)
-		(pin "29"
-		)
-		(pin "37"
-		)
-		(pin "40"
-		)
-		(pin "MP"
-		)
-		(pin "39"
-		)
-		(pin "33"
-		)
-		(pin "34"
-		)
-		(pin "35"
-		)
-		(pin "36"
-		)
-		(pin "32"
-		)
-		(pin "38"
-		)
-		(instances
-			(project "Microphone board"
-				(path "/54b36551-a175-45db-a91c-236f7d72a35b/933df564-ce74-4453-93df-6ff071652f89"
-					(reference "J1")
-					(unit 1)
-				)
-			)
-		)
-	)
-	(symbol
 		(lib_id "Device:C")
 		(at 140.97 81.28 0)
@@
 	(symbol
 		(lib_id "power:GND")
-		(at 199.39 142.24 0)
+		(at 204.47 30.48 0)
 		(unit 1)
 		(body_style 1)
@@
 		(fields_autoplaced yes)
 		(property "Reference" "#PWR096"
-			(at 199.39 148.59 0)
+			(at 204.47 36.83 0)
 			(hide yes)
 			(show_name no)
@@
 		)
 		(property "Value" "GND"
-			(at 199.39 147.32 0)
+			(at 204.47 35.56 0)
 			(show_name no)
 			(do_not_autoplace no)
@@
 		)
 		(property "Footprint" ""
-			(at 199.39 142.24 0)
+			(at 204.47 30.48 0)
 			(hide yes)
 			(show_name no)
@@
 		)
 		(property "Datasheet" ""
-			(at 199.39 142.24 0)
+			(at 204.47 30.48 0)
 			(hide yes)
 			(show_name no)
@@
 		)
 		(property "Description" "Power symbol creates a global label with name \"GND\" , ground"
-			(at 199.39 142.24 0)
-			(hide yes)
-			(show_name no)
+			(at 204.47 30.48 0)
+			(hide yes)
+			(show_name no)

Commit message: finished r1 of the board
Parts:
- J1: footprint Connector_FFC-FPC:Amphenol_F32R-1A7x1-11040_1x40-1MP_P0.5mm_Horizontal -> Connector_FFC-FPC:Hirose_FH12-40S-0.5SH_1x40-1MP_P0.50mm_Horizontal
Connections:
- net GND: no longer J1.31 (Pin_31)
- new net FMC_NE1: J1.31 (Pin_31)
Changed lines of the file:
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@@
-	)
-	(junction
-		(at 191.77 58.42)
-		(diameter 0)
-		(color 0 0 0 0)
 	)
 	(junction
@@
 	)
 	(bus_entry
+		(at 176.53 55.88)
+		(size 2.54 2.54)
+		(stroke
+			(width 0)
+			(type default)
+		)
+	)
+	(bus_entry
 		(at 176.53 68.58)
 		(size 2.54 2.54)
@@
 	(wire
 		(pts
-			(xy 191.77 58.42) (xy 191.77 111.76)
-		)
-		(stroke
-			(width 0)
-			(type default)
-		)
-	)
-	(wire
-		(pts
-			(xy 191.77 55.88) (xy 191.77 58.42)
+			(xy 191.77 55.88) (xy 191.77 111.76)
 		)
 		(stroke
@@
 	(wire
 		(pts
-			(xy 191.77 58.42) (xy 194.31 58.42)
-		)
-		(stroke
-			(width 0)
-			(type default)
-		)
-	)
-	(wire
-		(pts
 			(xy 194.31 50.8) (xy 189.23 50.8)
 		)
@@
 		(pts
 			(xy 189.23 53.34) (xy 189.23 50.8)
+		)
+		(stroke
+			(width 0)
+			(type default)
+		)
+	)
+	(wire
+		(pts
+			(xy 179.07 58.42) (xy 194.31 58.42)
 		)
 		(stroke
@@
 	(label "FMC_D9"
 		(at 179.07 91.44 0)
+		(effects
+			(font
+				(size 1.27 1.27)
+			)
+			(justify left bottom)
+		)
+	)
+	(label "FMC_NE1"
+		(at 179.07 58.42 0)
 		(effects
 			(font
@@
 			)
 		)
-		(property "Footprint" "Connector_FFC-FPC:Amphenol_F32R-1A7x1-11040_1x40-1MP_P0.5mm_Horizontal"
+		(property "Footprint" "Connector_FFC-FPC:Hirose_FH12-40S-0.5SH_1x40-1MP_P0.50mm_Horizontal"
 			(at 199.39 86.36 0)
 			(hide yes)

Commit message: Updated project firmware
Parts:
- R39: footprint Resistor_SMD:R_0402_1005Metric -> Resistor_SMD:R_0603_1608Metric
Changed lines of the file:
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@@
 			)
 		)
-		(property "Footprint" "Resistor_SMD:R_0402_1005Metric"
+		(property "Footprint" "Resistor_SMD:R_0603_1608Metric"
 			(at 78.232 100.33 90)
 			(hide yes)
